Commit message: no gui

File: oz440_description/urdf/materials.xacro (robot description, xacro)
@@ -25,3 +25,15 @@
 	  <color rgba="1.0 1.0 1.0 1.0"/>
   	</material>
+    <material name="naio">
+        <texture filename="models://ground_plane/materials/textures/naio1.jpg" />
+    </material>
+    <!--<material name="Wheel_l">-->
+        <!--<texture filename="package://pr2_ogre/Media/materials/textures/pr2_wheel_left.png" />-->
+    <!--</material>-->
+    <!--<material name="Wheel_r">-->
+        <!--<texture filename="package://pr2_ogre/Media/materials/textures/pr2_wheel_right.png" />-->
+    <!--</material>-->
+    <!--<material name="RollLinks">-->
+        <!--<texture filename="package://pr2_ogre/Media/materials/textures/pr2_wheel_left.png" />-->
+    <!--</material>-->
 </robot>

File: oz440_description/urdf/oz440.xacro (robot description, xacro)
@@ -48,5 +48,5 @@
 				<box size="${chassis_top_length} ${chassis_top_width} ${chassis_top_height}"/>
 			</geometry>
-			<material name="white"/>
+			<material name="naio"/>
 		</visual>
 		<inertial>

Commit message: no material

File: oz440_description/urdf/materials.xacro (robot description, xacro)
@@ -25,7 +25,7 @@
 	  <color rgba="1.0 1.0 1.0 1.0"/>
   	</material>
-    <material name="naio">
-        <texture filename="models://ground_plane/materials/textures/naio1.jpg" />
-    </material>
+    <!--<material name="naio">-->
+        <!--<texture filename="models://ground_plane/materials/textures/naio1.jpg" />-->
+    <!--</material>-->
     <!--<material name="Wheel_l">-->
         <!--<texture filename="package://pr2_ogre/Media/materials/textures/pr2_wheel_left.png" />-->
