Commit message: white

File: oz440_description/urdf/oz440.xacro (robot description, xacro)
@@ -48,5 +48,5 @@
 				<box size="${chassis_top_length} ${chassis_top_width} ${chassis_top_height}"/>
 			</geometry>
-			<material name="naio"/>
+			<material name="white"/>
 		</visual>
 		<inertial>

Commit message: actuator friction?

File: oz440_description/urdf/oz440.xacro (robot description, xacro)
@@ -7,5 +7,5 @@
 	<xacro:include filename="$(find oz440_description)/urdf/macros.xacro" />
 	<!-- link de base, OBLIGATOIRE -->
-	<!--<link name="footprint" />-->
+	<link name="footprint" />
 	<!-- link pour la partie basse du chassis -->
 	<link name="chassis_bottom">
@@ -30,9 +30,9 @@
     </link>
     <!--&lt;!&ndash; joint liant footprint a la partie basse du chassis &ndash;&gt;-->
-    <!--<joint name="footprint_to_chassis_bottom_joint" type="fixed">-->
-		<!--<parent link="footprint"/>-->
-		<!--<child link="chassis_bottom"/>-->
-		<!--<origin rpy="0 0 0" xyz="0 0 0"/>-->
-    <!--</joint>-->
+    <joint name="footprint_to_chassis_bottom_joint" type="fixed">
+		<parent link="footprint"/>
+		<child link="chassis_bottom"/>
+		<origin rpy="0 0 0" xyz="0 0 0"/>
+    </joint>
 	<!-- link pour la partie haute du chassis -->
 	<link name="chassis_top">
