Commit message: side_drive working

File: oz440_description/urdf/macros.xacro (robot description, xacro)
@@ -60,5 +60,5 @@
       <origin xyz="${tX*wheels_spacing/2} ${tY*((chassis_bottom_width/2)+wheel_chassis_bottom_spacing+(wheel_width/2))} ${wheel_transmission_height-chassis_bottom_height/2}" rpy="0 0 0" />
       <axis xyz="0 1 0" rpy="0 0 0" />
-      <limit effort="50" velocity="3.4"/>
+      <limit effort="22" velocity="3.4"/>
       <joint_properties damping="0.0" friction="0.0"/>
     </joint>

Commit message: Sliding stoped

File: oz440_description/urdf/macros.xacro (robot description, xacro)
@@ -48,8 +48,8 @@
     </link>
     <gazebo reference="${fb}_${lr}_wheel">
-      <mu1 value="0.2"/>
-      <mu2 value="0.2"/>
+      <mu1 value="0.75"/>
+      <mu2 value="0.8"/>
       <kp  value="10000000.0" />
-      <kd  value="10.0" />
+      <kd  value="1.0" />
       <fdir1 value="0 0 0"/>
       <material>Gazebo/Black</material>
@@ -60,5 +60,5 @@
       <origin xyz="${tX*wheels_spacing/2} ${tY*((chassis_bottom_width/2)+wheel_chassis_bottom_spacing+(wheel_width/2))} ${wheel_transmission_height-chassis_bottom_height/2}" rpy="0 0 0" />
       <axis xyz="0 1 0" rpy="0 0 0" />
-      <limit effort="22" velocity="3.4"/>
+      <limit effort="100" velocity="100"/>
       <joint_properties damping="0.0" friction="0.0"/>
     </joint>

Commit message: heightmap and real speed

File: oz440_description/urdf/macros.xacro (robot description, xacro)
@@ -48,7 +48,7 @@
     </link>
     <gazebo reference="${fb}_${lr}_wheel">
-      <mu1 value="0.75"/>
-      <mu2 value="0.8"/>
-      <kp  value="10000000.0" />
+      <mu1 value="0.9"/>
+      <mu2 value="0.9"/>
+      <kp  value="5000000.0" />
       <kd  value="1.0" />
       <fdir1 value="0 0 0"/>
@@ -60,5 +60,5 @@
       <origin xyz="${tX*wheels_spacing/2} ${tY*((chassis_bottom_width/2)+wheel_chassis_bottom_spacing+(wheel_width/2))} ${wheel_transmission_height-chassis_bottom_height/2}" rpy="0 0 0" />
       <axis xyz="0 1 0" rpy="0 0 0" />
-      <limit effort="100" velocity="100"/>
+      <limit effort="200" velocity="3.4"/>
       <joint_properties damping="0.0" friction="0.0"/>
     </joint>

Commit message: Color ground _ grass and rocks maps

File: oz440_description/urdf/macros.xacro (robot description, xacro)
@@ -6,6 +6,6 @@
   <xacro:macro name="cylinder_inertia" params="m r h">
     <inertia  ixx="${m*(3*r*r+h*h)/12}" ixy = "0" ixz = "0"
-      iyy="${m*(3*r*r+h*h)/12}" iyz = "0"
-      izz="${m*r*r/2}"
+              iyy="${m*(3*r*r+h*h)/12}" iyz = "0"
+              izz="${m*r*r/2}"
     />
   </xacro:macro>
@@ -13,6 +13,6 @@
   <xacro:macro name="box_inertia" params="m x y z">
     <inertia  ixx="${m*(y*y+z*z)/12}" ixy = "0" ixz = "0"
-      iyy="${m*(x*x+z*z)/12}" iyz = "0"
-      izz="${m*(x*x+z*z)/12}"
+              iyy="${m*(x*x+z*z)/12}" iyz = "0"
+              izz="${m*(x*x+z*z)/12}"
     />
   </xacro:macro>
@@ -20,6 +20,6 @@
   <xacro:macro name="sphere_inertia" params="m r">
     <inertia  ixx="${2*m*r*r/5}" ixy = "0" ixz = "0"
-      iyy="${2*m*r*r/5}" iyz = "0"
-      izz="${2*m*r*r/5}"
+              iyy="${2*m*r*r/5}" iyz = "0"
+              izz="${2*m*r*r/5}"
     />
   </xacro:macro>
@@ -31,15 +31,17 @@
         <geometry>
           <cylinder length="${wheel_width}" radius="${wheel_diameter/2}"/>
-        </geometry>
-      </collision>
-      <visual>
-        <origin xyz="0 0 0" rpy="0 ${PI/2} ${PI/2}" />
-        <geometry>
-          <cylinder length="${wheel_width}" radius="${wheel_diameter/2}"/>
+          <!--<mesh filename="/home/fanny/.gazebo/models/Wheel/roue.dae "/>-->
+        </geometry>
+      </collision>
+      <visual>
+        <origin xyz="0 0 0" rpy="0 ${PI/2} 0" />
+        <geometry>
+          <!--<cylinder length="${wheel_width}" radius="${wheel_diameter/2}"/>-->
+          <mesh filename="/home/fanny/.gazebo/models/Wheel/roue.dae "/>
         </geometry>
         <material name="black"/>
       </visual>
       <inertial>
-        <origin xyz="0 0 0" rpy="0 ${PI/2} ${PI/2}" />
+        <origin xyz="0 0 0" rpy="0 ${PI/2} 0" />
         <mass value="${wheel_mass}"/>
         <cylinder_inertia m="${wheel_mass}" r="${wheel_diameter/2}" h="${wheel_width}"/>
@@ -48,7 +50,7 @@
     </link>
     <gazebo reference="${fb}_${lr}_wheel">
-      <mu1 value="0.9"/>
-      <mu2 value="0.9"/>
-      <kp  value="5000000.0" />
+      <mu1 value="0.99"/>
+      <mu2 value="0.99"/>
+      <kp  value="1e+7" />
       <kd  value="1.0" />
       <fdir1 value="0 0 0"/>
@@ -78,19 +80,19 @@
     <link name="actuator_base_link">
       <inertial>
-          <mass value="1"/>
-          <origin xyz="0 0 0" rpy="0 0 0"/>
-          <box_inertia m="${actuator_base_Mass}" x="${actuator_base_Length}" y="${actuator_base_Width}" z="${actuator_base_Height}"/>
+        <mass value="1"/>
+        <origin xyz="0 0 0" rpy="0 0 0"/>
+        <box_inertia m="${actuator_base_Mass}" x="${actuator_base_Length}" y="${actuator_base_Width}" z="${actuator_base_Height}"/>
       </inertial>
       <collision name="collision_actuator">
-          <origin xyz="0 0 0" rpy="0 0 0"/>
-          <geometry>
-            <box size="${actuator_base_Length} ${actuator_base_Width} ${actuator_base_Height}"/>
-          </geometry>
-      </collision>
-      <visual>
         <origin xyz="0 0 0" rpy="0 0 0"/>
         <geometry>
           <box size="${actuator_base_Length} ${actuator_base_Width} ${actuator_base_Height}"/>
         </geometry>
+      </collision>
+      <visual>
+        <origin xyz="0 0 0" rpy="0 0 0"/>
+        <geometry>
+          <box size="${actuator_base_Length} ${actuator_base_Width} ${actuator_base_Height}"/>
+        </geometry>
         <material name="green"/>
       </visual>
@@ -98,19 +100,19 @@
     <link name="actuator_part1_link">
       <inertial>
-          <mass value="1"/>
-          <origin xyz="0 0 0" rpy="0 0 0"/>
-          <box_inertia m="${actuator_part1_Mass}" x="${actuator_part1_Length}" y="${actuator_part1_Width}" z="${actuator_part1_Height}"/>
+        <mass value="1"/>
+        <origin xyz="0 0 0" rpy="0 0 0"/>
+        <box_inertia m="${actuator_part1_Mass}" x="${actuator_part1_Length}" y="${actuator_part1_Width}" z="${actuator_part1_Height}"/>
       </inertial>
       <collision name="collision_actuator">
-          <origin xyz="0 0 0" rpy="0 0 0"/>
-          <geometry>
-            <box size="${actuator_part1_Length} ${actuator_part1_Width} ${actuator_part1_Height}"/>
-          </geometry>
-      </collision>
-      <visual>
         <origin xyz="0 0 0" rpy="0 0 0"/>
         <geometry>
           <box size="${actuator_part1_Length} ${actuator_part1_Width} ${actuator_part1_Height}"/>
         </geometry>
+      </collision>
+      <visual>
+        <origin xyz="0 0 0" rpy="0 0 0"/>
+        <geometry>
+          <box size="${actuator_part1_Length} ${actuator_part1_Width} ${actuator_part1_Height}"/>
+        </geometry>
         <material name="green"/>
       </visual>
@@ -118,13 +120,13 @@
     <link name="actuator_part2_link">
       <inertial>
-          <mass value="1"/>
-          <origin xyz="0 0 0" rpy="0 0 0"/>
-          <box_inertia m="${actuator_part2_Mass}" x="${actuator_part2_Length}" y="${actuator_part2_Width}" z="${actuator_part2_Height}"/>
+        <mass value="1"/>
+        <origin xyz="0 0 0" rpy="0 0 0"/>
+        <box_inertia m="${actuator_part2_Mass}" x="${actuator_part2_Length}" y="${actuator_part2_Width}" z="${actuator_part2_Height}"/>
       </inertial>
       <collision name="collision_actuator">
-          <origin xyz="0 0 0" rpy="0 0 0"/>
-          <geometry>
-            <box size="${actuator_part2_Length} ${actuator_part2_Width} ${actuator_part2_Height}"/>
-          </geometry>
+        <origin xyz="0 0 0" rpy="0 0 0"/>
+        <geometry>
+          <box size="${actuator_part2_Length} ${actuator_part2_Width} ${actuator_part2_Height}"/>
+        </geometry>
       </collision>
       <visual>
@@ -146,5 +148,5 @@
       <origin xyz="${-actuator_base_Length/2-actuator_part1_Length/2} 0 ${actuator_base_Height/2}" rpy="0 0 0"/>
       <axis rpy="0 0 0" xyz="0 0 -1"/>
-      <limit upper="0.0" lower=".15" effort="1" velocity=".1"/>
+      <limit upper="0.15" lower="0.15" effort="1" velocity="0.1"/>
     </joint>
     <joint name="actuator_part1_to_actuator_part2_joint" type="fixed">
@@ -198,7 +200,7 @@
       </visual>
       <inertial>
-          <mass value="1"/>
-          <origin xyz="0 0 0" rpy="0 0 0"/>
-          <box_inertia m="${lidar_Mass}" x="${lidar_Lenght}" y="${lidar_Width}" z="${lidar_Height}"/>
+        <mass value="1"/>
+        <origin xyz="0 0 0" rpy="0 0 0"/>
+        <box_inertia m="${lidar_Mass}" x="${lidar_Lenght}" y="${lidar_Width}" z="${lidar_Height}"/>
       </inertial>
     </link>
@@ -225,7 +227,7 @@
       </visual>
       <inertial>
-          <mass value="1"/>
-          <origin xyz="0 0 0" rpy="0 0 0"/>
-          <box_inertia m="${IMU_base_Mass}" x="${IMU_base_Length}" y="${IMU_base_Width}" z="${IMU_base_Height}"/>
+        <mass value="1"/>
+        <origin xyz="0 0 0" rpy="0 0 0"/>
+        <box_inertia m="${IMU_base_Mass}" x="${IMU_base_Length}" y="${IMU_base_Width}" z="${IMU_base_Height}"/>
       </inertial>
     </link>
@@ -244,7 +246,7 @@
       </visual>
       <inertial>
-          <mass value="1"/>
-          <origin xyz="0 0 0" rpy="0 0 0"/>
-          <box_inertia m="${IMU_Mass}" x="${IMU_Length}" y="${IMU_Width}" z="${IMU_Height}"/>
+        <mass value="1"/>
+        <origin xyz="0 0 0" rpy="0 0 0"/>
+        <box_inertia m="${IMU_Mass}" x="${IMU_Length}" y="${IMU_Width}" z="${IMU_Height}"/>
       </inertial>
     </link>
@@ -276,7 +278,7 @@
       </visual>
       <inertial>
-          <mass value="1"/>
-          <origin xyz="0 0 0" rpy="0 0 0"/>
-          <box_inertia m="${bumper_base_Mass}" x="${bumper_base_Length}" y="${bumper_base_Width}" z="${bumper_base_Height}"/>
+        <mass value="1"/>
+        <origin xyz="0 0 0" rpy="0 0 0"/>
+        <box_inertia m="${bumper_base_Mass}" x="${bumper_base_Length}" y="${bumper_base_Width}" z="${bumper_base_Height}"/>
       </inertial>
     </link>
@@ -295,7 +297,7 @@
       </visual>
       <inertial>
-          <mass value="1"/>
-          <origin xyz="0 0 0" rpy="0 0 0"/>
-          <box_inertia m="${bumper_Mass}" x="${bumper_Length}" y="${bumper_Width}" z="${bumper_Height}"/>
+        <mass value="1"/>
+        <origin xyz="0 0 0" rpy="0 0 0"/>
+        <box_inertia m="${bumper_Mass}" x="${bumper_Length}" y="${bumper_Width}" z="${bumper_Height}"/>
       </inertial>
     </link>

Commit message: v1.0

File: oz440_description/urdf/macros.xacro (robot description, xacro)
@@ -31,5 +31,4 @@
         <geometry>
           <cylinder length="${wheel_width}" radius="${wheel_diameter/2}"/>
-          <!--<mesh filename="/home/fanny/.gazebo/models/Wheel/roue.dae "/>-->
         </geometry>
       </collision>
@@ -37,6 +36,5 @@
         <origin xyz="0 0 0" rpy="0 ${PI/2} 0" />
         <geometry>
-          <!--<cylinder length="${wheel_width}" radius="${wheel_diameter/2}"/>-->
-          <mesh filename="/home/fanny/.gazebo/models/Wheel/roue.dae "/>
+          <mesh filename="model:///Wheel/roue.dae "/>
         </geometry>
         <material name="black"/>

Commit message: with models

File: oz440_description/urdf/macros.xacro (robot description, xacro)
@@ -36,5 +36,5 @@
         <origin xyz="0 0 0" rpy="0 ${PI/2} 0" />
         <geometry>
-          <mesh filename="model:///Wheel/roue.dae "/>
+          <mesh filename="model://Wheel/roue.dae "/>
         </geometry>
         <material name="black"/>

Commit message: level world

File: oz440_description/urdf/macros.xacro (robot description, xacro)
@@ -70,5 +70,5 @@
       <actuator name="${fb}_${lr}_Motor">
         <hardwareInterface>EffortJointInterface</hardwareInterface>
-        <mechanicalReduction>46</mechanicalReduction>
+        <mechanicalRedu.ction>46</mechanicalRedu.ction>
       </actuator>
     </transmission>

File: oz440_description/urdf/materials.xacro (robot description, xacro)
@@ -25,15 +25,3 @@
 	  <color rgba="1.0 1.0 1.0 1.0"/>
   	</material>
-    <!--<material name="naio">-->
-        <!--<texture filename="models://ground_plane/materials/textures/naio1.jpg" />-->
-    <!--</material>-->
-    <!--<material name="Wheel_l">-->
-        <!--<texture filename="package://pr2_ogre/Media/materials/textures/pr2_wheel_left.png" />-->
-    <!--</material>-->
-    <!--<material name="Wheel_r">-->
-        <!--<texture filename="package://pr2_ogre/Media/materials/textures/pr2_wheel_right.png" />-->
-    <!--</material>-->
-    <!--<material name="RollLinks">-->
-        <!--<texture filename="package://pr2_ogre/Media/materials/textures/pr2_wheel_left.png" />-->
-    <!--</material>-->
 </robot>

Commit message: actuator

File: oz440_description/urdf/macros.xacro (robot description, xacro)
@@ -28,18 +28,27 @@
     <link name="${fb}_${lr}_wheel">
       <collision>
+        <!--<origin xyz="0 0 0" rpy="0 ${PI/2} 0" />-->
+        <origin xyz="${wheel_diameter/2} -${wheel_width/2} -${wheel_diameter/2}" rpy="0 0 ${PI/2}" />
+        <geometry>
+          <!--<cylinder length="${wheel_width}" radius="${wheel_diameter/2}"/>-->
+          <mesh filename="model://Wheel/pneu.dae" scale ="0.001 0.001 0.001" />
+        </geometry>
+      </collision>
+      <visual>
         <origin xyz="0 0 0" rpy="0 ${PI/2} ${PI/2}" />
         <geometry>
-          <cylinder length="${wheel_width}" radius="${wheel_diameter/2}"/>
-        </geometry>
-      </collision>
-      <visual>
-        <origin xyz="0 0 0" rpy="0 ${PI/2} 0" />
-        <geometry>
-          <mesh filename="model://Wheel/roue.dae "/>
+          <cylinder length="${wheel_width}" radius="${wheel_diameter/4}"/>
+        </geometry>
+      </visual>
+      <visual>
+        <origin xyz="${wheel_diameter/2} -${wheel_width/2} -${wheel_diameter/2}" rpy="0 0 ${PI/2}" />
+        <geometry>
+          <mesh filename="model://Wheel/pneu.dae" scale ="0.001 0.001 0.001" />
         </geometry>
         <material name="black"/>
       </visual>
       <inertial>
-        <origin xyz="0 0 0" rpy="0 ${PI/2} 0" />
+        <origin xyz="0 0 0" rpy="${PI/2} 0 ${PI/2}" />
+        <!--<origin xyz="0 0 0" rpy="0 ${PI/2} 0" />-->
         <mass value="${wheel_mass}"/>
         <cylinder_inertia m="${wheel_mass}" r="${wheel_diameter/2}" h="${wheel_width}"/>
@@ -96,4 +105,12 @@
       </visual>
     </link>
+    <gazebo reference="actuator_base_link">
+      <mu1 value="0.99"/>
+      <mu2 value="0.99"/>
+      <kp  value="1e+7" />
+      <kd  value="1.0" />
+      <fdir1 value="0 0 0"/>
+      <material>Gazebo/Green</material>
+    </gazebo>
     <link name="actuator_part1_link">
       <inertial>
@@ -116,4 +133,12 @@
       </visual>
     </link>
+    <gazebo reference="actuator_part1_link">
+      <mu1 value="0.99"/>
+      <mu2 value="0.99"/>
+      <kp  value="1e+7" />
+      <kd  value="1.0" />
+      <fdir1 value="0 0 0"/>
+      <material>Gazebo/Green</material>
+    </gazebo>
     <link name="actuator_part2_link">
       <inertial>
@@ -136,4 +161,12 @@
       </visual>
     </link>
+    <gazebo reference="actuator_part2_link">
+      <mu1 value="0.99"/>
+      <mu2 value="0.99"/>
+      <kp  value="1e+7" />
+      <kd  value="1.0" />
+      <fdir1 value="0 0 0"/>
+      <material>Gazebo/Green</material>
+    </gazebo>
     <joint name="chassis_bottom_to_actuator_base_joint" type="fixed">
       <parent link="${parent}"/>
@@ -145,7 +178,17 @@
       <child link="actuator_part1_link"/>
       <origin xyz="${-actuator_base_Length/2-actuator_part1_Length/2} 0 ${actuator_base_Height/2}" rpy="0 0 0"/>
-      <axis rpy="0 0 0" xyz="0 0 -1"/>
-      <limit upper="0.15" lower="0.15" effort="1" velocity="0.1"/>
-    </joint>
+      <axis rpy="0 0 0" xyz="0 0 1"/>
+      <limit upper="0" lower="-0.15" effort="1" velocity="0.1"/>
+    </joint>
+    <transmission name="actuator_base_link_to_actuator_part1_trans">
+      <type>transmission_interface/SimpleTransmission</type>
+      <joint name="actuator_base_link_to_actuator_part1_joint">
+        <hardwareInterface>EffortJointInterface</hardwareInterface>
+      </joint>
+      <actuator name="actuator_base_link_to_actuator_part1_actuator">
+        <hardwareInterface>EffortJointInterface</hardwareInterface>
+        <mechanicalRedu.ction>46</mechanicalRedu.ction>
+      </actuator>
+    </transmission>
     <joint name="actuator_part1_to_actuator_part2_joint" type="fixed">
       <parent link="actuator_part1_link"/>
@@ -176,4 +219,12 @@
       </inertial>
     </link>
+    <gazebo reference="camera_stereo_link">
+      <mu1 value="0.99"/>
+      <mu2 value="0.99"/>
+      <kp  value="1e+7" />
+      <kd  value="1.0" />
+      <fdir1 value="0 0 0"/>
+      <material>Gazebo/Grey</material>
+    </gazebo>
     <joint name="chassis_top_to_camera_stereo" type="fixed">
       <parent link="${parent}"/>
@@ -230,4 +281,12 @@
       </inertial>
     </link>
+    <gazebo reference="IMU_base_link">
+      <mu1 value="0.99"/>
+      <mu2 value="0.99"/>
+      <kp  value="1e+7" />
+      <kd  value="1.0" />
+      <fdir1 value="0 0 0"/>
+      <material>Gazebo/Green</material>
+    </gazebo>
     <link name="IMU_link">
       <collision>
@@ -249,4 +308,12 @@
       </inertial>
     </link>
+    <gazebo reference="IMU_link">
+      <mu1 value="0.99"/>
+      <mu2 value="0.99"/>
+      <kp  value="1e+7" />
+      <kd  value="1.0" />
+      <fdir1 value="0 0 0"/>
+      <material>Gazebo/Grey</material>
+    </gazebo>
     <joint name="actuator_base_to_IMU_base_joint" type="fixed">
       <parent link="${parent}"/>

File: oz440_description/urdf/materials.xacro (robot description, xacro)
@@ -2,5 +2,5 @@
 <robot>
 	<material name="black">
-	  <color rgba="0.0 0.0 0.0 1.0"/>
+	  <color rgba="0.02 0.02 0.02 1.0"/>
 	</material>
 	<material name="blue">

File: oz440_description/urdf/properties.xacro (robot description, xacro)
@@ -23,15 +23,15 @@
 	<xacro:property name="actuator_base_Mass" value="1"/>
 	<xacro:property name="actuator_base_Length" value="0.04"/>
-	<xacro:property name="actuator_base_Width" value="0.2"/>
-	<xacro:property name="actuator_base_Height" value="0.4"/>
+	<xacro:property name="actuator_base_Width" value="0.1"/>
+	<xacro:property name="actuator_base_Height" value="0.2"/>
 	<xacro:property name="actuator_base_chassis_spacing" value="0.02"/>
 	<xacro:property name="actuator_part1_Mass" value="1"/>
-	<xacro:property name="actuator_part1_Length" value="0.22"/>
-	<xacro:property name="actuator_part1_Width" value="0.22"/>
-	<xacro:property name="actuator_part1_Height" value="0.15"/>
+	<xacro:property name="actuator_part1_Length" value="0.1"/>
+	<xacro:property name="actuator_part1_Width" value="0.07"/>
+	<xacro:property name="actuator_part1_Height" value="0.1"/>
 	<xacro:property name="actuator_part2_Mass" value="1"/>
-	<xacro:property name="actuator_part2_Length" value="0.22"/>
-	<xacro:property name="actuator_part2_Width" value="0.4"/>
-	<xacro:property name="actuator_part2_Height" value="0.04"/>
+	<xacro:property name="actuator_part2_Length" value="0.1"/>
+	<xacro:property name="actuator_part2_Width" value="0.12"/>
+	<xacro:property name="actuator_part2_Height" value="0.02"/>
 	<!-- Proprietes de la camera -->
 	<xacro:property name="cameraSizeX" value="0.075"/>

Commit message: wheel

File: oz440_description/urdf/macros.xacro (robot description, xacro)
@@ -167,5 +167,5 @@
       <kd  value="1.0" />
       <fdir1 value="0 0 0"/>
-      <material>Gazebo/Green</material>
+      <material>Gazebo/Grass</material>
     </gazebo>
     <joint name="chassis_bottom_to_actuator_base_joint" type="fixed">

Commit message: grass green

File: oz440_description/urdf/macros.xacro (robot description, xacro)
@@ -111,5 +111,5 @@
       <kd  value="1.0" />
       <fdir1 value="0 0 0"/>
-      <material>Gazebo/Green</material>
+      <material>Gazebo/Grass</material>
     </gazebo>
     <link name="actuator_part1_link">
@@ -139,5 +139,5 @@
       <kd  value="1.0" />
       <fdir1 value="0 0 0"/>
-      <material>Gazebo/Green</material>
+      <material>Gazebo/Grass</material>
     </gazebo>
     <link name="actuator_part2_link">

Commit message: fix actuator 4

File: oz440_description/urdf/macros.xacro (robot description, xacro)
@@ -111,5 +111,7 @@
       <kd  value="1.0" />
       <fdir1 value="0 0 0"/>
-      <material>Gazebo/Grass</material>
+      <material name="orange">
+        <color rgba="${255/255} ${108/255} ${10/255} 1.0"/>
+      </material>
     </gazebo>
     <link name="actuator_part1_link">

Commit message: fixed?

File: oz440_description/urdf/macros.xacro (robot description, xacro)
@@ -28,9 +28,9 @@
     <link name="${fb}_${lr}_wheel">
       <collision>
-        <!--<origin xyz="0 0 0" rpy="0 ${PI/2} 0" />-->
-        <origin xyz="${wheel_diameter/2} -${wheel_width/2} -${wheel_diameter/2}" rpy="0 0 ${PI/2}" />
-        <geometry>
-          <!--<cylinder length="${wheel_width}" radius="${wheel_diameter/2}"/>-->
-          <mesh filename="model://Wheel/pneu.dae" scale ="0.001 0.001 0.001" />
+        <origin xyz="0 0 0" rpy="0 ${PI/2} 0" />
+        <!--<origin xyz="${wheel_diameter/2} -${wheel_width/2} -${wheel_diameter/2}" rpy="0 0 ${PI/2}" />-->
+        <geometry>
+          <cylinder length="${wheel_width}" radius="${wheel_diameter/2}"/>
+          <!--<mesh filename="model://Wheel/pneu.dae" scale ="0.001 0.001 0.001" />-->
         </geometry>
       </collision>
@@ -111,7 +111,5 @@
       <kd  value="1.0" />
       <fdir1 value="0 0 0"/>
-      <material name="orange">
-        <color rgba="${255/255} ${108/255} ${10/255} 1.0"/>
-      </material>
+      <material> Gazebo/white </material>
     </gazebo>
     <link name="actuator_part1_link">

Commit message: fixed?

File: oz440_description/urdf/macros.xacro (robot description, xacro)
@@ -28,5 +28,5 @@
     <link name="${fb}_${lr}_wheel">
       <collision>
-        <origin xyz="0 0 0" rpy="0 ${PI/2} 0" />
+        <origin xyz="0 0 0" rpy="0 ${PI/2} ${PI/2}" />
         <!--<origin xyz="${wheel_diameter/2} -${wheel_width/2} -${wheel_diameter/2}" rpy="0 0 ${PI/2}" />-->
         <geometry>
