Commit message: fixed?

File: oz440_description/urdf/macros.xacro (robot description, xacro)
@@ -35,14 +35,19 @@
         </geometry>
       </collision>
+      <!--<visual>-->
+        <!--<origin xyz="0 0 0" rpy="0 ${PI/2} ${PI/2}" />-->
+        <!--<geometry>-->
+          <!--<cylinder length="${wheel_width}" radius="${wheel_diameter/4}"/>-->
+        <!--</geometry>-->
+      <!--</visual>-->
       <visual>
         <origin xyz="0 0 0" rpy="0 ${PI/2} ${PI/2}" />
-        <geometry>
-          <cylinder length="${wheel_width}" radius="${wheel_diameter/4}"/>
-        </geometry>
-      </visual>
-      <visual>
-        <origin xyz="${wheel_diameter/2} -${wheel_width/2} -${wheel_diameter/2}" rpy="0 0 ${PI/2}" />
-        <geometry>
-          <mesh filename="model://Wheel/pneu.dae" scale ="0.001 0.001 0.001" />
+        <!--<origin xyz="${wheel_diameter/2} -${wheel_width/2} -${wheel_diameter/2}" rpy="0 0 ${PI/2}" />-->
+        <geometry>
+        <cylinder length="${wheel_width}" radius="${wheel_diameter/2}"/>
+        <!--<mesh filename="model://Wheel/pneu.dae" scale ="0.001 0.001 0.001" />-->
+        <!--<origin xyz="${wheel_diameter/2} -${wheel_width/2} -${wheel_diameter/2}" rpy="0 0 ${PI/2}" />-->
+        <!--<geometry>-->
+          <!--<mesh filename="model://Wheel/pneu.dae" scale ="0.001 0.001 0.001" />-->
         </geometry>
         <material name="black"/>

Commit message: tool

File: oz440_description/urdf/macros.xacro (robot description, xacro)
@@ -202,4 +202,56 @@
     </joint>
   </xacro:macro>
+  <!-- macro pour l'outils -->
+  <xacro:macro name="tool_macro" params="parent">
+    <link name="tool">
+      <inertial>
+        <mass value="100"/>
+        <origin xyz="-0.15 0 0" rpy="0 0 0"/>
+        <sphere_inertia m="50" r="0.05"/>
+      </inertial>
+      <collision name="sphere">
+        <origin xyz="-0.15 0 0" rpy="0 0 0"/>
+        <geometry>
+          <sphere radius="0.05"/>
+        </geometry>
+      </collision>
+      <visual>
+        <origin xyz="-0.15 0 0" rpy="0 0 0"/>
+        <geometry>
+          <sphere radius="0.05"/>
+        </geometry>
+        <material name="grey"/>
+      </visual>
+      <!--<collision name="stick">-->
+        <!--<origin xyz="-0.05 0 0" rpy="0 ${PI/2} 0"/>-->
+        <!--<geometry>-->
+          <!--<cylinder radius="0.01" length="0.1"/>-->
+        <!--</geometry>-->
+      <!--</collision>-->
+      <visual>
+        <origin xyz="-0.05 0 0" rpy="0 ${PI/2} 0"/>
+        <geometry>
+          <cylinder radius="0.01" length="0.1"/>
+        </geometry>
+        <material name="grey"/>
+      </visual>
+    </link>
+    <gazebo reference="tool">
+      <mu1 value="0.999"/>
+      <mu2 value="0.999"/>
+      <kp  value="1e+7" />
+      <kd  value="1.0" />
+      <fdir1 value="0 0 0"/>
+      <material> Gazebo/Grey </material>
+    </gazebo>
+    <joint name="tool_to_actuator_part_2" type="continuous">
+      <parent link="actuator_part2_link"/>
+      <child link="tool"/>
+      <origin xyz="0 0 ${-actuator_part2_Height/2}" rpy="0 0 0" />
+      <axis xyz="0 1 0" rpy="0 0 0" />
+      <limit effort="50" velocity="3"/>
+      <joint_properties damping="0.0" friction="0.3"/>
+    </joint>
+  </xacro:macro>
   <!-- macro pour la camera stereo -->
   <xacro:macro name="camera_stereo" params="parent">

File: oz440_description/urdf/oz440.xacro (robot description, xacro)
@@ -77,3 +77,4 @@
 	<!-- inclusion du bumper -->
 	<bumper parent="chassis_top"/>
+	<tool_macro parent="actuator_part2_link"/>
 </robot>

File: oz440_description/urdf/properties.xacro (robot description, xacro)
@@ -31,7 +31,7 @@
 	<xacro:property name="actuator_part1_Height" value="0.1"/>
 	<xacro:property name="actuator_part2_Mass" value="1"/>
-	<xacro:property name="actuator_part2_Length" value="0.1"/>
-	<xacro:property name="actuator_part2_Width" value="0.12"/>
-	<xacro:property name="actuator_part2_Height" value="0.02"/>
+	<xacro:property name="actuator_part2_Length" value="0.04"/>
+	<xacro:property name="actuator_part2_Width" value="0.04"/>
+	<xacro:property name="actuator_part2_Height" value="0.04"/>
 	<!-- Proprietes de la camera -->
 	<xacro:property name="cameraSizeX" value="0.075"/>

Commit message: tool fix 1

File: oz440_description/urdf/macros.xacro (robot description, xacro)
@@ -250,6 +250,6 @@
       <origin xyz="0 0 ${-actuator_part2_Height/2}" rpy="0 0 0" />
       <axis xyz="0 1 0" rpy="0 0 0" />
-      <limit effort="50" velocity="3"/>
-      <joint_properties damping="0.0" friction="0.3"/>
+      <limit effort="100" velocity="5"/>
+      <joint_properties damping="0.0" friction="0.2"/>
     </joint>
   </xacro:macro>

Commit message: tool fix 2

File: oz440_description/urdf/macros.xacro (robot description, xacro)
@@ -206,5 +206,5 @@
     <link name="tool">
       <inertial>
-        <mass value="100"/>
+        <mass value="50"/>
         <origin xyz="-0.15 0 0" rpy="0 0 0"/>
         <sphere_inertia m="50" r="0.05"/>
@@ -238,6 +238,6 @@
     </link>
     <gazebo reference="tool">
-      <mu1 value="0.999"/>
-      <mu2 value="0.999"/>
+      <mu1 value="0.99"/>
+      <mu2 value="0.99"/>
       <kp  value="1e+7" />
       <kd  value="1.0" />
@@ -250,6 +250,6 @@
       <origin xyz="0 0 ${-actuator_part2_Height/2}" rpy="0 0 0" />
       <axis xyz="0 1 0" rpy="0 0 0" />
-      <limit effort="100" velocity="5"/>
-      <joint_properties damping="0.0" friction="0.2"/>
+      <limit effort="200" velocity="10"/>
+      <joint_properties damping="0.0" friction="0.0"/>
     </joint>
   </xacro:macro>

Commit message: vid

File: oz440_description/urdf/macros.xacro (robot description, xacro)
@@ -118,4 +118,31 @@
       <material> Gazebo/white </material>
     </gazebo>
+    <link name="butee">
+      <inertial>
+        <mass value="0.01"/>
+        <origin xyz="${-actuator_base_Length/2 - 0.01} 0 ${actuator_base_Height/2 - actuator_part1_Height/2 - 0.01}" rpy="0 0 0"/>
+        <box_inertia m="0.01" x="0.02" y="${actuator_base_Width}" z="0.02"/>
+      </inertial>
+      <collision name="butee">
+        <origin xyz="${-actuator_base_Length/2 - 0.01} 0 ${actuator_base_Height/2 - actuator_part1_Height/2 - 0.01}" rpy="0 0 0"/>
+        <geometry>
+          <box size="0.02 ${actuator_base_Width} 0.02"/>
+        </geometry>
+      </collision>
+      <visual>
+        <origin xyz="${-actuator_base_Length/2 - 0.01} 0 ${actuator_base_Height/2 - actuator_part1_Height/2 - 0.01}" rpy="0 0 0"/>
+        <geometry>
+          <box size="0.02 ${actuator_base_Width} 0.02"/>
+        </geometry>
+      </visual>
+    </link>
+    <gazebo reference="butee">
+      <mu1 value="0.99"/>
+      <mu2 value="0.99"/>
+      <kp  value="1e+7" />
+      <kd  value="1.0" />
+      <fdir1 value="0 0 0"/>
+      <material> Gazebo/white </material>
+    </gazebo>
     <link name="actuator_part1_link">
       <inertial>
@@ -178,4 +205,9 @@
       <child link="actuator_base_link"/>
       <origin xyz="${-chassis_bottom_length/2-actuator_base_Length/2-actuator_base_chassis_spacing} 0 ${chassis_bottom_height/2}" rpy="0 0 0"/>
+    </joint>
+    <joint name="butee_to_actuator_base_joint" type="fixed">
+      <parent link="actuator_base_link"/>
+      <child link="butee"/>
+      <origin xyz="0 0 -0.01" rpy="0 0 0"/>
     </joint>
     <joint name="actuator_base_link_to_actuator_part1_joint" type="prismatic">
@@ -184,5 +216,5 @@
       <origin xyz="${-actuator_base_Length/2-actuator_part1_Length/2} 0 ${actuator_base_Height/2}" rpy="0 0 0"/>
       <axis rpy="0 0 0" xyz="0 0 1"/>
-      <limit upper="0" lower="-0.15" effort="1" velocity="0.1"/>
+      <limit upper="0" lower="-0.15" effort="10" velocity="0"/>
     </joint>
     <transmission name="actuator_base_link_to_actuator_part1_trans">
@@ -206,8 +238,15 @@
     <link name="tool">
       <inertial>
-        <mass value="50"/>
-        <origin xyz="-0.15 0 0" rpy="0 0 0"/>
-        <sphere_inertia m="1" r="0.05"/>
-      </inertial>
+        <origin xyz="-0.15 0 0" rpy="0 0 0" />
+        <!--<origin xyz="0 0 0" rpy="0 ${PI/2} 0" />-->
+        <mass value="${10}"/>
+        <sphere_inertia m="${10}" r="${0.01}"/>
+      </inertial>
+      <gravity>1</gravity>
+      <!--<inertial>-->
+        <!--<mass value="7.5" />-->
+        <!--<origin xyz="-0.15 0 0" rpy="0 0 0"/>-->
+        <!--<inertia ixx="1e-3" ixy="0" ixz="0" iyy="1e-3" iyz="0" izz="1e-3" />-->
+      <!--</inertial>-->
       <collision name="sphere">
         <origin xyz="-0.15 0 0" rpy="0 0 0"/>
@@ -250,5 +289,5 @@
       <origin xyz="0 0 ${-actuator_part2_Height/2}" rpy="0 0 0" />
       <axis xyz="0 1 0" rpy="0 0 0" />
-      <limit effort="200" velocity="10"/>
+      <dynamics damping="0.0"/>
       <joint_properties damping="0.0" friction="0.0"/>
     </joint>

File: oz440_description/urdf/oz440.xacro (robot description, xacro)
@@ -64,4 +64,5 @@
 	<!-- inclusion du porte outils -->
     <actuator_macro parent="chassis_bottom"/>
+	<!--<tool_macro parent="actuator_part2_link"/>-->
     <!-- inclusion des roues -->
 	<wheel fb="front" lr="right" tX="1" tY="-1"/>
@@ -77,4 +78,3 @@
 	<!-- inclusion du bumper -->
 	<bumper parent="chassis_top"/>
-	<tool_macro parent="actuator_part2_link"/>
 </robot>

Commit message: vid

File: oz440_description/urdf/macros.xacro (robot description, xacro)
@@ -42,9 +42,9 @@
       <!--</visual>-->
       <visual>
-        <origin xyz="0 0 0" rpy="0 ${PI/2} ${PI/2}" />
-        <!--<origin xyz="${wheel_diameter/2} -${wheel_width/2} -${wheel_diameter/2}" rpy="0 0 ${PI/2}" />-->
-        <geometry>
-        <cylinder length="${wheel_width}" radius="${wheel_diameter/2}"/>
-        <!--<mesh filename="model://Wheel/pneu.dae" scale ="0.001 0.001 0.001" />-->
+        <!--<origin xyz="0 0 0" rpy="0 ${PI/2} ${PI/2}" />-->
+        <origin xyz="${wheel_diameter/2} -${wheel_width/2} -${wheel_diameter/2}" rpy="0 0 ${PI/2}" />
+        <geometry>
+        <!--<cylinder length="${wheel_width}" radius="${wheel_diameter/2}"/>-->
+          <mesh filename="model://Wheel/pneu.dae" scale ="0.001 0.001 0.001" />
         <!--<origin xyz="${wheel_diameter/2} -${wheel_width/2} -${wheel_diameter/2}" rpy="0 0 ${PI/2}" />-->
         <!--<geometry>-->
@@ -118,31 +118,31 @@
       <material> Gazebo/white </material>
     </gazebo>
-    <link name="butee">
-      <inertial>
-        <mass value="0.01"/>
-        <origin xyz="${-actuator_base_Length/2 - 0.01} 0 ${actuator_base_Height/2 - actuator_part1_Height/2 - 0.01}" rpy="0 0 0"/>
-        <box_inertia m="0.01" x="0.02" y="${actuator_base_Width}" z="0.02"/>
-      </inertial>
-      <collision name="butee">
-        <origin xyz="${-actuator_base_Length/2 - 0.01} 0 ${actuator_base_Height/2 - actuator_part1_Height/2 - 0.01}" rpy="0 0 0"/>
-        <geometry>
-          <box size="0.02 ${actuator_base_Width} 0.02"/>
-        </geometry>
-      </collision>
-      <visual>
-        <origin xyz="${-actuator_base_Length/2 - 0.01} 0 ${actuator_base_Height/2 - actuator_part1_Height/2 - 0.01}" rpy="0 0 0"/>
-        <geometry>
-          <box size="0.02 ${actuator_base_Width} 0.02"/>
-        </geometry>
-      </visual>
-    </link>
-    <gazebo reference="butee">
-      <mu1 value="0.99"/>
-      <mu2 value="0.99"/>
-      <kp  value="1e+7" />
-      <kd  value="1.0" />
-      <fdir1 value="0 0 0"/>
-      <material> Gazebo/white </material>
-    </gazebo>
+    <!--<link name="butee">-->
+      <!--<inertial>-->
+        <!--<mass value="0.01"/>-->
+        <!--<origin xyz="${-actuator_base_Length/2 - 0.01} 0 ${actuator_base_Height/2 - actuator_part1_Height/2 - 0.01}" rpy="0 0 0"/>-->
+        <!--<box_inertia m="0.01" x="0.02" y="${actuator_base_Width}" z="0.02"/>-->
+      <!--</inertial>-->
+      <!--<collision name="butee">-->
+        <!--<origin xyz="${-actuator_base_Length/2 - 0.01} 0 ${actuator_base_Height/2 - actuator_part1_Height/2 - 0.01}" rpy="0 0 0"/>-->
+        <!--<geometry>-->
+          <!--<box size="0.02 ${actuator_base_Width} 0.02"/>-->
+        <!--</geometry>-->
+      <!--</collision>-->
+      <!--<visual>-->
+        <!--<origin xyz="${-actuator_base_Length/2 - 0.01} 0 ${actuator_base_Height/2 - actuator_part1_Height/2 - 0.01}" rpy="0 0 0"/>-->
+        <!--<geometry>-->
+          <!--<box size="0.02 ${actuator_base_Width} 0.02"/>-->
+        <!--</geometry>-->
+      <!--</visual>-->
+    <!--</link>-->
+    <!--<gazebo reference="butee">-->
+      <!--<mu1 value="0.99"/>-->
+      <!--<mu2 value="0.99"/>-->
+      <!--<kp  value="1e+7" />-->
+      <!--<kd  value="1.0" />-->
+      <!--<fdir1 value="0 0 0"/>-->
+      <!--<material> Gazebo/white </material>-->
+    <!--</gazebo>-->
     <link name="actuator_part1_link">
       <inertial>
@@ -206,9 +206,9 @@
       <origin xyz="${-chassis_bottom_length/2-actuator_base_Length/2-actuator_base_chassis_spacing} 0 ${chassis_bottom_height/2}" rpy="0 0 0"/>
     </joint>
-    <joint name="butee_to_actuator_base_joint" type="fixed">
-      <parent link="actuator_base_link"/>
-      <child link="butee"/>
-      <origin xyz="0 0 -0.01" rpy="0 0 0"/>
-    </joint>
+    <!--<joint name="butee_to_actuator_base_joint" type="fixed">-->
+      <!--<parent link="actuator_base_link"/>-->
+      <!--<child link="butee"/>-->
+      <!--<origin xyz="0 0 -0.01" rpy="0 0 0"/>-->
+    <!--</joint>-->
     <joint name="actuator_base_link_to_actuator_part1_joint" type="prismatic">
       <parent link="actuator_base_link"/>
@@ -238,27 +238,20 @@
     <link name="tool">
       <inertial>
-        <origin xyz="-0.15 0 0" rpy="0 0 0" />
-        <!--<origin xyz="0 0 0" rpy="0 ${PI/2} 0" />-->
-        <mass value="${10}"/>
-        <sphere_inertia m="${10}" r="${0.01}"/>
+        <origin xyz="0 0 -0.013" rpy="0 0 0" />
+        <mass value="10"/>
+        <sphere_inertia m="${10}" r="${0.05}"/>
       </inertial>
       <gravity>1</gravity>
-      <!--<inertial>-->
-        <!--<mass value="7.5" />-->
-        <!--<origin xyz="-0.15 0 0" rpy="0 0 0"/>-->
-        <!--<inertia ixx="1e-3" ixy="0" ixz="0" iyy="1e-3" iyz="0" izz="1e-3" />-->
-      <!--</inertial>-->
       <collision name="sphere">
-        <origin xyz="-0.15 0 0" rpy="0 0 0"/>
-        <geometry>
-          <sphere radius="0.05"/>
-        </geometry>
-      </collision>
-      <visual>
-        <origin xyz="-0.15 0 0" rpy="0 0 0"/>
-        <geometry>
-          <sphere radius="0.05"/>
-        </geometry>
-        <material name="grey"/>
+        <origin xyz="0 0 -0.013" rpy="0 0 0"/>
+        <geometry>
+          <sphere radius="0.03"/>
+        </geometry>
+      </collision>
+      <visual>
+        <origin xyz="0 0 -0.013" rpy="0 0 0"/>
+        <geometry>
+          <sphere radius="0.03"/>
+        </geometry>
       </visual>
       <!--<collision name="stick">-->
@@ -269,9 +262,8 @@
       <!--</collision>-->
       <visual>
-        <origin xyz="-0.05 0 0" rpy="0 ${PI/2} 0"/>
+        <origin xyz="0 0 -0.05" rpy="0 0 0"/>
         <geometry>
           <cylinder radius="0.01" length="0.1"/>
         </geometry>
-        <material name="grey"/>
       </visual>
     </link>
@@ -284,11 +276,16 @@
       <material> Gazebo/Grey </material>
     </gazebo>
-    <joint name="tool_to_actuator_part_2" type="continuous">
+    <!--<joint name="tool_to_actuator_part_2" type="continuous">-->
+      <!--<parent link="actuator_part2_link"/>-->
+      <!--<child link="tool"/>-->
+      <!--<origin xyz="0 0 ${-actuator_part2_Height/2}" rpy="0 0 0" />-->
+      <!--<axis xyz="0 1 0" rpy="0 0 0" />-->
+      <!--<dynamics damping="0.0"/>-->
+      <!--<joint_properties damping="0.0" friction="0.0"/>-->
+    <!--</joint>-->
+    <joint name="tool_to_actuator_part_2" type="fixed">
       <parent link="actuator_part2_link"/>
       <child link="tool"/>
-      <origin xyz="0 0 ${-actuator_part2_Height/2}" rpy="0 0 0" />
-      <axis xyz="0 1 0" rpy="0 0 0" />
-      <dynamics damping="0.0"/>
-      <joint_properties damping="0.0" friction="0.0"/>
+      <origin rpy="0 0 ${-actuator_part2_Height/2}" xyz="0 0 0"/>
     </joint>
   </xacro:macro>

File: oz440_description/urdf/properties.xacro (robot description, xacro)
@@ -27,10 +27,10 @@
 	<xacro:property name="actuator_base_chassis_spacing" value="0.02"/>
 	<xacro:property name="actuator_part1_Mass" value="1"/>
-	<xacro:property name="actuator_part1_Length" value="0.1"/>
-	<xacro:property name="actuator_part1_Width" value="0.07"/>
+	<xacro:property name="actuator_part1_Length" value="0.2"/>
+	<xacro:property name="actuator_part1_Width" value="0.1"/>
 	<xacro:property name="actuator_part1_Height" value="0.1"/>
 	<xacro:property name="actuator_part2_Mass" value="1"/>
-	<xacro:property name="actuator_part2_Length" value="0.04"/>
-	<xacro:property name="actuator_part2_Width" value="0.04"/>
+	<xacro:property name="actuator_part2_Length" value="0.07"/>
+	<xacro:property name="actuator_part2_Width" value="0.07"/>
 	<xacro:property name="actuator_part2_Height" value="0.04"/>
 	<!-- Proprietes de la camera -->

Commit message: actuator fix

File: oz440_description/urdf/macros.xacro (robot description, xacro)
@@ -45,9 +45,6 @@
         <origin xyz="${wheel_diameter/2} -${wheel_width/2} -${wheel_diameter/2}" rpy="0 0 ${PI/2}" />
         <geometry>
-        <!--<cylinder length="${wheel_width}" radius="${wheel_diameter/2}"/>-->
+          <!--<cylinder length="${wheel_width}" radius="${wheel_diameter/2}"/>-->
           <mesh filename="model://Wheel/pneu.dae" scale ="0.001 0.001 0.001" />
-        <!--<origin xyz="${wheel_diameter/2} -${wheel_width/2} -${wheel_diameter/2}" rpy="0 0 ${PI/2}" />-->
-        <!--<geometry>-->
-          <!--<mesh filename="model://Wheel/pneu.dae" scale ="0.001 0.001 0.001" />-->
         </geometry>
         <material name="black"/>
@@ -62,6 +59,6 @@
     </link>
     <gazebo reference="${fb}_${lr}_wheel">
-      <mu1 value="0.99"/>
-      <mu2 value="0.99"/>
+      <mu1 value="0.999"/>
+      <mu2 value="0.999"/>
       <kp  value="1e+7" />
       <kd  value="1.0" />
@@ -74,5 +71,5 @@
       <origin xyz="${tX*wheels_spacing/2} ${tY*((chassis_bottom_width/2)+wheel_chassis_bottom_spacing+(wheel_width/2))} ${wheel_transmission_height-chassis_bottom_height/2}" rpy="0 0 0" />
       <axis xyz="0 1 0" rpy="0 0 0" />
-      <limit effort="200" velocity="3.4"/>
+      <limit effort="2000" velocity="3.4"/>
       <joint_properties damping="0.0" friction="0.0"/>
     </joint>
@@ -118,31 +115,4 @@
       <material> Gazebo/white </material>
     </gazebo>
-    <!--<link name="butee">-->
-      <!--<inertial>-->
-        <!--<mass value="0.01"/>-->
-        <!--<origin xyz="${-actuator_base_Length/2 - 0.01} 0 ${actuator_base_Height/2 - actuator_part1_Height/2 - 0.01}" rpy="0 0 0"/>-->
-        <!--<box_inertia m="0.01" x="0.02" y="${actuator_base_Width}" z="0.02"/>-->
-      <!--</inertial>-->
-      <!--<collision name="butee">-->
-        <!--<origin xyz="${-actuator_base_Length/2 - 0.01} 0 ${actuator_base_Height/2 - actuator_part1_Height/2 - 0.01}" rpy="0 0 0"/>-->
-        <!--<geometry>-->
-          <!--<box size="0.02 ${actuator_base_Width} 0.02"/>-->
-        <!--</geometry>-->
-      <!--</collision>-->
-      <!--<visual>-->
-        <!--<origin xyz="${-actuator_base_Length/2 - 0.01} 0 ${actuator_base_Height/2 - actuator_part1_Height/2 - 0.01}" rpy="0 0 0"/>-->
-        <!--<geometry>-->
-          <!--<box size="0.02 ${actuator_base_Width} 0.02"/>-->
-        <!--</geometry>-->
-      <!--</visual>-->
-    <!--</link>-->
-    <!--<gazebo reference="butee">-->
-      <!--<mu1 value="0.99"/>-->
-      <!--<mu2 value="0.99"/>-->
-      <!--<kp  value="1e+7" />-->
-      <!--<kd  value="1.0" />-->
-      <!--<fdir1 value="0 0 0"/>-->
-      <!--<material> Gazebo/white </material>-->
-    <!--</gazebo>-->
     <link name="actuator_part1_link">
       <inertial>
@@ -206,9 +176,4 @@
       <origin xyz="${-chassis_bottom_length/2-actuator_base_Length/2-actuator_base_chassis_spacing} 0 ${chassis_bottom_height/2}" rpy="0 0 0"/>
     </joint>
-    <!--<joint name="butee_to_actuator_base_joint" type="fixed">-->
-      <!--<parent link="actuator_base_link"/>-->
-      <!--<child link="butee"/>-->
-      <!--<origin xyz="0 0 -0.01" rpy="0 0 0"/>-->
-    <!--</joint>-->
     <joint name="actuator_base_link_to_actuator_part1_joint" type="prismatic">
       <parent link="actuator_base_link"/>
@@ -238,19 +203,19 @@
     <link name="tool">
       <inertial>
-        <origin xyz="0 0 -0.013" rpy="0 0 0" />
-        <mass value="10"/>
-        <sphere_inertia m="${10}" r="${0.05}"/>
+        <origin xyz="0 0 -0.017" rpy="0 0 0" />
+        <mass value="40"/>
+        <sphere_inertia m="${40}" r="${0.05}"/>
       </inertial>
       <gravity>1</gravity>
       <collision name="sphere">
-        <origin xyz="0 0 -0.013" rpy="0 0 0"/>
-        <geometry>
-          <sphere radius="0.03"/>
-        </geometry>
-      </collision>
-      <visual>
-        <origin xyz="0 0 -0.013" rpy="0 0 0"/>
-        <geometry>
-          <sphere radius="0.03"/>
+        <origin xyz="0 0 -0.17" rpy="0 0 0"/>
+        <geometry>
+          <sphere radius="0.06"/>
+        </geometry>
+      </collision>
+      <visual>
+        <origin xyz="0 0 -0.17" rpy="0 0 0"/>
+        <geometry>
+          <sphere radius="0.06"/>
         </geometry>
       </visual>
@@ -262,7 +227,7 @@
       <!--</collision>-->
       <visual>
-        <origin xyz="0 0 -0.05" rpy="0 0 0"/>
-        <geometry>
-          <cylinder radius="0.01" length="0.1"/>
+        <origin xyz="0 0 -0.065" rpy="0 0 0"/>
+        <geometry>
+          <cylinder radius="0.01" length="0.13"/>
         </geometry>
       </visual>

File: oz440_description/urdf/oz440.xacro (robot description, xacro)
@@ -64,5 +64,5 @@
 	<!-- inclusion du porte outils -->
     <actuator_macro parent="chassis_bottom"/>
-	<!--<tool_macro parent="actuator_part2_link"/>-->
+	<tool_macro parent="actuator_part2_link"/>
     <!-- inclusion des roues -->
 	<wheel fb="front" lr="right" tX="1" tY="-1"/>

File: oz440_description/urdf/properties.xacro (robot description, xacro)
@@ -27,10 +27,10 @@
 	<xacro:property name="actuator_base_chassis_spacing" value="0.02"/>
 	<xacro:property name="actuator_part1_Mass" value="1"/>
-	<xacro:property name="actuator_part1_Length" value="0.2"/>
-	<xacro:property name="actuator_part1_Width" value="0.1"/>
+	<xacro:property name="actuator_part1_Length" value="0.1"/>
+	<xacro:property name="actuator_part1_Width" value="0.15"/>
 	<xacro:property name="actuator_part1_Height" value="0.1"/>
 	<xacro:property name="actuator_part2_Mass" value="1"/>
-	<xacro:property name="actuator_part2_Length" value="0.07"/>
-	<xacro:property name="actuator_part2_Width" value="0.07"/>
+	<xacro:property name="actuator_part2_Length" value="0.04"/>
+	<xacro:property name="actuator_part2_Width" value="0.04"/>
 	<xacro:property name="actuator_part2_Height" value="0.04"/>
 	<!-- Proprietes de la camera -->
