Commit message: actuator fix lighter

File: oz440_description/urdf/macros.xacro (robot description, xacro)
@@ -42,9 +42,9 @@
       <!--</visual>-->
       <visual>
-        <!--<origin xyz="0 0 0" rpy="0 ${PI/2} ${PI/2}" />-->
-        <origin xyz="${wheel_diameter/2} -${wheel_width/2} -${wheel_diameter/2}" rpy="0 0 ${PI/2}" />
-        <geometry>
-          <!--<cylinder length="${wheel_width}" radius="${wheel_diameter/2}"/>-->
-          <mesh filename="model://Wheel/pneu.dae" scale ="0.001 0.001 0.001" />
+        <origin xyz="0 0 0" rpy="0 ${PI/2} ${PI/2}" />
+        <!--<origin xyz="${wheel_diameter/2} -${wheel_width/2} -${wheel_diameter/2}" rpy="0 0 ${PI/2}" />-->
+        <geometry>
+          <cylinder length="${wheel_width}" radius="${wheel_diameter/2}"/>
+          <!--<mesh filename="model://Wheel/pneu.dae" scale ="0.001 0.001 0.001" />-->
         </geometry>
         <material name="black"/>
@@ -204,6 +204,6 @@
       <inertial>
         <origin xyz="0 0 -0.017" rpy="0 0 0" />
-        <mass value="40"/>
-        <sphere_inertia m="${40}" r="${0.05}"/>
+        <mass value="20"/>
+        <sphere_inertia m="${20}" r="${0.05}"/>
       </inertial>
       <gravity>1</gravity>
@@ -234,6 +234,6 @@
     </link>
     <gazebo reference="tool">
-      <mu1 value="0.99"/>
-      <mu2 value="0.99"/>
+      <mu1 value="0.1"/>
+      <mu2 value="0.1"/>
       <kp  value="1e+7" />
       <kd  value="1.0" />

Commit message: actuator fix lighter

File: oz440_description/urdf/macros.xacro (robot description, xacro)
@@ -204,6 +204,6 @@
       <inertial>
         <origin xyz="0 0 -0.017" rpy="0 0 0" />
-        <mass value="20"/>
-        <sphere_inertia m="${20}" r="${0.05}"/>
+        <mass value="10"/>
+        <sphere_inertia m="${10}" r="${0.05}"/>
       </inertial>
       <gravity>1</gravity>

Commit message: actuator fix lighter

File: oz440_description/urdf/macros.xacro (robot description, xacro)
@@ -204,6 +204,6 @@
       <inertial>
         <origin xyz="0 0 -0.017" rpy="0 0 0" />
-        <mass value="10"/>
-        <sphere_inertia m="${10}" r="${0.05}"/>
+        <mass value="1"/>
+        <sphere_inertia m="${1}" r="${0.05}"/>
       </inertial>
       <gravity>1</gravity>

Commit message: actuator 2

File: oz440_description/urdf/macros.xacro (robot description, xacro)
@@ -176,4 +176,9 @@
       <origin xyz="${-chassis_bottom_length/2-actuator_base_Length/2-actuator_base_chassis_spacing} 0 ${chassis_bottom_height/2}" rpy="0 0 0"/>
     </joint>
+    <!--<joint name="actuator_base_link_to_actuator_part1_joint" type="fixed">-->
+      <!--<parent link="actuator_base_link"/>-->
+      <!--<child link="actuator_part1_link"/>-->
+      <!--<origin xyz="${-actuator_base_Length/2-actuator_part1_Length/2} 0 ${actuator_base_Height/2}" rpy="0 0 0"/>-->
+    <!--</joint>-->
     <joint name="actuator_base_link_to_actuator_part1_joint" type="prismatic">
       <parent link="actuator_base_link"/>
@@ -181,16 +186,16 @@
       <origin xyz="${-actuator_base_Length/2-actuator_part1_Length/2} 0 ${actuator_base_Height/2}" rpy="0 0 0"/>
       <axis rpy="0 0 0" xyz="0 0 1"/>
-      <limit upper="0" lower="-0.15" effort="10" velocity="0"/>
-    </joint>
-    <transmission name="actuator_base_link_to_actuator_part1_trans">
-      <type>transmission_interface/SimpleTransmission</type>
-      <joint name="actuator_base_link_to_actuator_part1_joint">
-        <hardwareInterface>EffortJointInterface</hardwareInterface>
-      </joint>
-      <actuator name="actuator_base_link_to_actuator_part1_actuator">
-        <hardwareInterface>EffortJointInterface</hardwareInterface>
-        <mechanicalRedu.ction>46</mechanicalRedu.ction>
-      </actuator>
-    </transmission>
+      <limit upper="0" lower="-0.01" effort="100" velocity="3"/>
+    </joint>
+    <!--<transmission name="actuator_base_link_to_actuator_part1_trans">-->
+      <!--<type>transmission_interface/SimpleTransmission</type>-->
+      <!--<joint name="actuator_base_link_to_actuator_part1_joint">-->
+        <!--<hardwareInterface>EffortJointInterface</hardwareInterface>-->
+      <!--</joint>-->
+      <!--<actuator name="actuator_base_link_to_actuator_part1_actuator">-->
+        <!--<hardwareInterface>EffortJointInterface</hardwareInterface>-->
+        <!--<mechanicalRedu.ction>46</mechanicalRedu.ction>-->
+      <!--</actuator>-->
+    <!--</transmission>-->
     <joint name="actuator_part1_to_actuator_part2_joint" type="fixed">
       <parent link="actuator_part1_link"/>
@@ -220,10 +225,4 @@
         </geometry>
       </visual>
-      <!--<collision name="stick">-->
-        <!--<origin xyz="-0.05 0 0" rpy="0 ${PI/2} 0"/>-->
-        <!--<geometry>-->
-          <!--<cylinder radius="0.01" length="0.1"/>-->
-        <!--</geometry>-->
-      <!--</collision>-->
       <visual>
         <origin xyz="0 0 -0.065" rpy="0 0 0"/>

Commit message: actuator 2

File: oz440_description/urdf/macros.xacro (robot description, xacro)
@@ -186,5 +186,5 @@
       <origin xyz="${-actuator_base_Length/2-actuator_part1_Length/2} 0 ${actuator_base_Height/2}" rpy="0 0 0"/>
       <axis rpy="0 0 0" xyz="0 0 1"/>
-      <limit upper="0" lower="-0.01" effort="100" velocity="3"/>
+      <limit upper="0" lower="-0.015" effort="100" velocity="3"/>
     </joint>
     <!--<transmission name="actuator_base_link_to_actuator_part1_trans">-->

Commit message: actuator friction?

File: oz440_description/urdf/macros.xacro (robot description, xacro)
@@ -51,17 +51,15 @@
       </visual>
       <inertial>
-        <origin xyz="0 0 0" rpy="${PI/2} 0 ${PI/2}" />
-        <!--<origin xyz="0 0 0" rpy="0 ${PI/2} 0" />-->
+        <origin xyz="0 0 0" rpy="0 ${PI/2} ${PI/2}" />
         <mass value="${wheel_mass}"/>
         <cylinder_inertia m="${wheel_mass}" r="${wheel_diameter/2}" h="${wheel_width}"/>
       </inertial>
-      <gravity>1</gravity>
     </link>
     <gazebo reference="${fb}_${lr}_wheel">
-      <mu1 value="0.99"/>
-      <mu2 value="0.99"/>
-      <kp  value="1e+7" />
-      <kd  value="1.0" />
-      <fdir1 value="0 0 0"/>
+      <gravity>true</gravity>
+      <mu1 value="0.99"/>
+      <mu2 value="0.99"/>
+      <kp  value="1e+6" />
+      <kd  value="1.0" />
       <material>Gazebo/Black</material>
     </gazebo>
@@ -71,6 +69,5 @@
       <origin xyz="${tX*wheels_spacing/2} ${tY*((chassis_bottom_width/2)+wheel_chassis_bottom_spacing+(wheel_width/2))} ${wheel_transmission_height-chassis_bottom_height/2}" rpy="0 0 0" />
       <axis xyz="0 1 0" rpy="0 0 0" />
-      <limit effort="2000" velocity="3.4"/>
-      <joint_properties damping="0.0" friction="0.0"/>
+      <dynamics damping="0.1" friction="0.0"/>
     </joint>
     <transmission name="${fb}_${lr}_trans">
@@ -104,5 +101,4 @@
           <box size="${actuator_base_Length} ${actuator_base_Width} ${actuator_base_Height}"/>
         </geometry>
-        <material name="green"/>
       </visual>
     </link>
@@ -117,5 +113,5 @@
     <link name="actuator_part1_link">
       <inertial>
-        <mass value="1"/>
+        <mass value="${actuator_part1_Mass}"/>
         <origin xyz="0 0 0" rpy="0 0 0"/>
         <box_inertia m="${actuator_part1_Mass}" x="${actuator_part1_Length}" y="${actuator_part1_Width}" z="${actuator_part1_Height}"/>
@@ -132,5 +128,4 @@
           <box size="${actuator_part1_Length} ${actuator_part1_Width} ${actuator_part1_Height}"/>
         </geometry>
-        <material name="green"/>
       </visual>
     </link>
@@ -141,9 +136,9 @@
       <kd  value="1.0" />
       <fdir1 value="0 0 0"/>
-      <material>Gazebo/Grass</material>
+      <material>Gazebo/Green</material>
     </gazebo>
     <link name="actuator_part2_link">
       <inertial>
-        <mass value="1"/>
+        <mass value="${actuator_part2_Mass}"/>
         <origin xyz="0 0 0" rpy="0 0 0"/>
         <box_inertia m="${actuator_part2_Mass}" x="${actuator_part2_Length}" y="${actuator_part2_Width}" z="${actuator_part2_Height}"/>
@@ -160,5 +155,4 @@
           <box size="${actuator_part2_Length} ${actuator_part2_Width} ${actuator_part2_Height}"/>
         </geometry>
-        <material name="green"/>
       </visual>
     </link>
@@ -169,5 +163,5 @@
       <kd  value="1.0" />
       <fdir1 value="0 0 0"/>
-      <material>Gazebo/Grass</material>
+      <material>Gazebo/Green</material>
     </gazebo>
     <joint name="chassis_bottom_to_actuator_base_joint" type="fixed">
@@ -176,9 +170,4 @@
       <origin xyz="${-chassis_bottom_length/2-actuator_base_Length/2-actuator_base_chassis_spacing} 0 ${chassis_bottom_height/2}" rpy="0 0 0"/>
     </joint>
-    <!--<joint name="actuator_base_link_to_actuator_part1_joint" type="fixed">-->
-      <!--<parent link="actuator_base_link"/>-->
-      <!--<child link="actuator_part1_link"/>-->
-      <!--<origin xyz="${-actuator_base_Length/2-actuator_part1_Length/2} 0 ${actuator_base_Height/2}" rpy="0 0 0"/>-->
-    <!--</joint>-->
     <joint name="actuator_base_link_to_actuator_part1_joint" type="prismatic">
       <parent link="actuator_base_link"/>
@@ -186,16 +175,7 @@
       <origin xyz="${-actuator_base_Length/2-actuator_part1_Length/2} 0 ${actuator_base_Height/2}" rpy="0 0 0"/>
       <axis rpy="0 0 0" xyz="0 0 1"/>
-      <limit upper="0" lower="-0.015" effort="100" velocity="3"/>
-    </joint>
-    <!--<transmission name="actuator_base_link_to_actuator_part1_trans">-->
-      <!--<type>transmission_interface/SimpleTransmission</type>-->
-      <!--<joint name="actuator_base_link_to_actuator_part1_joint">-->
-        <!--<hardwareInterface>EffortJointInterface</hardwareInterface>-->
-      <!--</joint>-->
-      <!--<actuator name="actuator_base_link_to_actuator_part1_actuator">-->
-        <!--<hardwareInterface>EffortJointInterface</hardwareInterface>-->
-        <!--<mechanicalRedu.ction>46</mechanicalRedu.ction>-->
-      <!--</actuator>-->
-    <!--</transmission>-->
+      <limit upper="0" lower="-0.15" effort="100" velocity="1"/>
+      <dynamics damping="0.7" friction="0.9"/>
+    </joint>
     <joint name="actuator_part1_to_actuator_part2_joint" type="fixed">
       <parent link="actuator_part1_link"/>
@@ -233,19 +213,11 @@
     </link>
     <gazebo reference="tool">
-      <mu1 value="1"/>
-      <mu2 value="1"/>
-      <kp  value="1e+7" />
+      <mu1 value="0.99"/>
+      <mu2 value="0.99"/>
+      <kp  value="1e+4" />
       <kd  value="1.0" />
       <fdir1 value="0 0 0"/>
       <material> Gazebo/Grey </material>
     </gazebo>
-    <!--<joint name="tool_to_actuator_part_2" type="continuous">-->
-      <!--<parent link="actuator_part2_link"/>-->
-      <!--<child link="tool"/>-->
-      <!--<origin xyz="0 0 ${-actuator_part2_Height/2}" rpy="0 0 0" />-->
-      <!--<axis xyz="0 1 0" rpy="0 0 0" />-->
-      <!--<dynamics damping="0.0"/>-->
-      <!--<joint_properties damping="0.0" friction="0.0"/>-->
-    <!--</joint>-->
     <joint name="tool_to_actuator_part_2" type="fixed">
       <parent link="actuator_part2_link"/>
@@ -268,5 +240,4 @@
           <box size="${cameraSizeX} ${cameraSizeY} ${cameraSizeZ}"/>
         </geometry>
-        <material name="white"/>
       </visual>
       <inertial>

File: oz440_description/urdf/oz440.xacro (robot description, xacro)
@@ -4,8 +4,8 @@
 	<xacro:include filename="$(find oz440_description)/urdf/properties.xacro" />
     <xacro:include filename="$(find oz440_description)/urdf/oz440.gazebo" />
-    <xacro:include filename="$(find oz440_description)/urdf/materials.xacro" />
+    <!--<xacro:include filename="$(find oz440_description)/urdf/materials.xacro" />-->
 	<xacro:include filename="$(find oz440_description)/urdf/macros.xacro" />
 	<!-- link de base, OBLIGATOIRE -->
-	<link name="footprint" />
+	<!--<link name="footprint" />-->
 	<!-- link pour la partie basse du chassis -->
 	<link name="chassis_bottom">
@@ -29,10 +29,10 @@
 		</inertial>
     </link>
-    <!-- joint liant footprint a la partie basse du chassis -->
-    <joint name="footprint_to_chassis_bottom_joint" type="fixed">
-		<parent link="footprint"/>
-		<child link="chassis_bottom"/>
-		<origin rpy="0 0 0" xyz="0 0 0"/>
-    </joint>
+    <!--&lt;!&ndash; joint liant footprint a la partie basse du chassis &ndash;&gt;-->
+    <!--<joint name="footprint_to_chassis_bottom_joint" type="fixed">-->
+		<!--<parent link="footprint"/>-->
+		<!--<child link="chassis_bottom"/>-->
+		<!--<origin rpy="0 0 0" xyz="0 0 0"/>-->
+    <!--</joint>-->
 	<!-- link pour la partie haute du chassis -->
 	<link name="chassis_top">
@@ -48,5 +48,4 @@
 				<box size="${chassis_top_length} ${chassis_top_width} ${chassis_top_height}"/>
 			</geometry>
-			<material name="white"/>
 		</visual>
 		<inertial>

Commit message: actuator friction?

File: oz440_description/urdf/macros.xacro (robot description, xacro)
@@ -178,4 +178,14 @@
       <dynamics damping="0.7" friction="0.9"/>
     </joint>
+    <transmission name="actuator_base_link_to_actuator_part1_trans">
+      <type>transmission_interface/SimpleTransmission</type>
+      <joint name="actuator_base_link_to_actuator_part1_joint">
+        <hardwareInterface>EffortJointInterface</hardwareInterface>
+      </joint>
+      <actuator name="actuator_base_link_to_actuator_part1_motor">
+        <hardwareInterface>EffortJointInterface</hardwareInterface>
+        <mechanicalRedu.ction>46</mechanicalRedu.ction>
+      </actuator>
+    </transmission>
     <joint name="actuator_part1_to_actuator_part2_joint" type="fixed">
       <parent link="actuator_part1_link"/>

Commit message: cool tool 1

File: oz440_description/urdf/macros.xacro (robot description, xacro)
@@ -138,5 +138,5 @@
       <material>Gazebo/Green</material>
     </gazebo>
-    <link name="actuator_part2_link">
+    <link name="actuator_part21_link">
       <inertial>
         <mass value="${actuator_part2_Mass}"/>
@@ -157,5 +157,59 @@
       </visual>
     </link>
-    <gazebo reference="actuator_part2_link">
+    <link name="actuator_part22_link">
+      <inertial>
+        <mass value="${actuator_part2_Mass}"/>
+        <origin xyz="0 0 0" rpy="0 0 0"/>
+        <box_inertia m="${actuator_part2_Mass}" x="${actuator_part2_Length}" y="${actuator_part2_Width}" z="${actuator_part2_Height}"/>
+      </inertial>
+      <collision name="collision_actuator">
+        <origin xyz="0 0 0" rpy="0 0 0"/>
+        <geometry>
+          <box size="${actuator_part2_Length} ${actuator_part2_Width} ${actuator_part2_Height}"/>
+        </geometry>
+      </collision>
+      <visual>
+        <origin xyz="0 0 0" rpy="0 0 0"/>
+        <geometry>
+          <box size="${actuator_part2_Length} ${actuator_part2_Width} ${actuator_part2_Height}"/>
+        </geometry>
+      </visual>
+    </link>
+    <link name="actuator_part23_link">
+      <inertial>
+        <mass value="${actuator_part2_Mass}"/>
+        <origin xyz="0 0 0" rpy="0 0 0"/>
+        <box_inertia m="${actuator_part2_Mass}" x="${actuator_part2_Length}" y="${actuator_part2_Width}" z="${actuator_part2_Height}"/>
+      </inertial>
+      <collision name="collision_actuator">
+        <origin xyz="0 0 0" rpy="0 0 0"/>
+        <geometry>
+          <box size="${actuator_part2_Length} ${actuator_part2_Width} ${actuator_part2_Height}"/>
+        </geometry>
+      </collision>
+      <visual>
+        <origin xyz="0 0 0" rpy="0 0 0"/>
+        <geometry>
+          <box size="${actuator_part2_Length} ${actuator_part2_Width} ${actuator_part2_Height}"/>
+        </geometry>
+      </visual>
+    </link>
+    <gazebo reference="actuator_part21_link">
+      <mu1 value="0.99"/>
+      <mu2 value="0.99"/>
+      <kp  value="1e+7" />
+      <kd  value="1.0" />
+      <fdir1 value="0 0 0"/>
+      <material>Gazebo/Green</material>
+    </gazebo>
+    <gazebo reference="actuator_part22_link">
+      <mu1 value="0.99"/>
+      <mu2 value="0.99"/>
+      <kp  value="1e+7" />
+      <kd  value="1.0" />
+      <fdir1 value="0 0 0"/>
+      <material>Gazebo/Green</material>
+    </gazebo>
+    <gazebo reference="actuator_part23_link">
       <mu1 value="0.99"/>
       <mu2 value="0.99"/>
@@ -188,39 +242,119 @@
       </actuator>
     </transmission>
-    <joint name="actuator_part1_to_actuator_part2_joint" type="fixed">
+    <joint name="actuator_part1_to_actuator_part21_joint" type="fixed">
       <parent link="actuator_part1_link"/>
-      <child link="actuator_part2_link"/>
+      <child link="actuator_part21_link"/>
       <origin xyz="0 0 ${-actuator_part1_Height/2-actuator_part2_Height/2}" rpy="0 0 0"/>
+    </joint>
+    <joint name="actuator_part1_to_actuator_part22_joint" type="fixed">
+      <parent link="actuator_part1_link"/>
+      <child link="actuator_part22_link"/>
+      <origin xyz="0 -0.18 ${-actuator_part1_Height/2-actuator_part2_Height/2}" rpy="0 0 0"/>
+    </joint>
+    <joint name="actuator_part1_to_actuator_part23_joint" type="fixed">
+      <parent link="actuator_part1_link"/>
+      <child link="actuator_part23_link"/>
+      <origin xyz="0 0.18 ${-actuator_part1_Height/2-actuator_part2_Height/2}" rpy="0 0 0"/>
     </joint>
   </xacro:macro>
   <!-- macro pour l'outils -->
   <xacro:macro name="tool_macro" params="parent">
-    <link name="tool">
-      <inertial>
-        <origin xyz="0 0 -0.017" rpy="0 0 0" />
-        <mass value="1"/>
-        <sphere_inertia m="${1}" r="${0.05}"/>
+    <link name="tool1">
+      <inertial>
+        <origin xyz="-0.25 0 -0.2" rpy="0 0 0" />
+        <mass value="10"/>
+        <sphere_inertia m="${10}" r="${0.05}"/>
       </inertial>
       <gravity>1</gravity>
       <collision name="sphere">
-        <origin xyz="0 0 -0.17" rpy="0 0 0"/>
-        <geometry>
-          <sphere radius="0.06"/>
-        </geometry>
-      </collision>
-      <visual>
-        <origin xyz="0 0 -0.17" rpy="0 0 0"/>
-        <geometry>
-          <sphere radius="0.06"/>
-        </geometry>
-      </visual>
-      <visual>
-        <origin xyz="0 0 -0.065" rpy="0 0 0"/>
-        <geometry>
-          <cylinder radius="0.01" length="0.13"/>
-        </geometry>
-      </visual>
-    </link>
-    <gazebo reference="tool">
+        <origin xyz="-0.25 0 -0.2" rpy="0 0 0"/>
+        <geometry>
+          <sphere radius="0.02"/>
+        </geometry>
+      </collision>
+      <visual>
+        <origin xyz="-0.25 0 -0.2" rpy="0 0 0"/>
+        <geometry>
+          <sphere radius="0.02"/>
+        </geometry>
+      </visual>
+      <visual>
+        <origin xyz="-0.125 0 -0.075" rpy="0 1.03 0"/>
+        <geometry>
+          <cylinder radius="0.007" length="0.29"/>
+        </geometry>
+      </visual>
+      <visual>
+        <origin xyz="-0.25 0 -0.165" rpy="0 0 0"/>
+        <geometry>
+          <cylinder radius="0.007" length="0.035"/>
+        </geometry>
+      </visual>
+    </link>
+    <link name="tool2">
+      <inertial>
+        <origin xyz="-0.25 -0.2 -0.2" rpy="0 0 0" />
+        <mass value="10"/>
+        <sphere_inertia m="${10}" r="${0.05}"/>
+      </inertial>
+      <gravity>1</gravity>
+      <collision name="sphere">
+        <origin xyz="-0.25 0 -0.2" rpy="0 0 0"/>
+        <geometry>
+          <sphere radius="0.02"/>
+        </geometry>
+      </collision>
+      <visual>
+        <origin xyz="-0.25 0 -0.2" rpy="0 0 0"/>
+        <geometry>
+          <sphere radius="0.02"/>
+        </geometry>
+      </visual>
+      <visual>
+        <origin xyz="-0.125 0 -0.075" rpy="0 1.03 0"/>
+        <geometry>
+          <cylinder radius="0.007" length="0.29"/>
+        </geometry>
+      </visual>
+      <visual>
+        <origin xyz="-0.25 0 -0.165" rpy="0 0 0"/>
+        <geometry>
+          <cylinder radius="0.007" length="0.035"/>
+        </geometry>
+      </visual>
+    </link>
+    <link name="tool3">
+      <inertial>
+        <origin xyz="-0.25 0 -0.2" rpy="0 0 0" />
+        <mass value="10"/>
+        <sphere_inertia m="${10}" r="${0.05}"/>
+      </inertial>
+      <gravity>1</gravity>
+      <collision name="sphere">
+        <origin xyz="-0.25 0 -0.2" rpy="0 0 0"/>
+        <geometry>
+          <sphere radius="0.02"/>
+        </geometry>
+      </collision>
+      <visual>
+        <origin xyz="-0.25 0 -0.2" rpy="0 0 0"/>
+        <geometry>
+          <sphere radius="0.02"/>
+        </geometry>
+      </visual>
+      <visual>
+        <origin xyz="-0.125 0 -0.075" rpy="0 1.03 0"/>
+        <geometry>
+          <cylinder radius="0.007" length="0.29"/>
+        </geometry>
+      </visual>
+      <visual>
+        <origin xyz="-0.25 0 -0.165" rpy="0 0 0"/>
+        <geometry>
+          <cylinder radius="0.007" length="0.035"/>
+        </geometry>
+      </visual>
+    </link>
+    <gazebo reference="tool1">
       <mu1 value="0.99"/>
       <mu2 value="0.99"/>
@@ -230,7 +364,33 @@
       <material> Gazebo/Grey </material>
     </gazebo>
-    <joint name="tool_to_actuator_part_2" type="fixed">
-      <parent link="actuator_part2_link"/>
-      <child link="tool"/>
+    <gazebo reference="tool2">
+      <mu1 value="0.99"/>
+      <mu2 value="0.99"/>
+      <kp  value="1e+4" />
+      <kd  value="1.0" />
+      <fdir1 value="0 0 0"/>
+      <material> Gazebo/Grey </material>
+    </gazebo>
+    <gazebo reference="tool3">
+      <mu1 value="0.99"/>
+      <mu2 value="0.99"/>
+      <kp  value="1e+4" />
+      <kd  value="1.0" />
+      <fdir1 value="0 0 0"/>
+      <material> Gazebo/Grey </material>
+    </gazebo>
+    <joint name="tool1_to_actuator_part_21" type="fixed">
+      <parent link="actuator_part21_link"/>
+      <child link="tool1"/>
+      <origin rpy="0 0 ${-actuator_part2_Height/2}" xyz="0 0 0"/>
+    </joint>
+    <joint name="tool2_to_actuator_part_22" type="fixed">
+      <parent link="actuator_part22_link"/>
+      <child link="tool2"/>
+      <origin rpy="0 0 ${-actuator_part2_Height/2}" xyz="0 0 0"/>
+    </joint>
+    <joint name="tool3_to_actuator_part_23" type="fixed">
+      <parent link="actuator_part23_link"/>
+      <child link="tool3"/>
       <origin rpy="0 0 ${-actuator_part2_Height/2}" xyz="0 0 0"/>
     </joint>

File: oz440_description/urdf/properties.xacro (robot description, xacro)
@@ -27,7 +27,7 @@
 	<xacro:property name="actuator_base_chassis_spacing" value="0.02"/>
 	<xacro:property name="actuator_part1_Mass" value="1"/>
-	<xacro:property name="actuator_part1_Length" value="0.1"/>
-	<xacro:property name="actuator_part1_Width" value="0.15"/>
-	<xacro:property name="actuator_part1_Height" value="0.1"/>
+	<xacro:property name="actuator_part1_Length" value="0.05"/>
+	<xacro:property name="actuator_part1_Width" value="0.41"/>
+	<xacro:property name="actuator_part1_Height" value="0.05"/>
 	<xacro:property name="actuator_part2_Mass" value="1"/>
 	<xacro:property name="actuator_part2_Length" value="0.04"/>
