Commit message: cool tool 1

File: oz440_description/urdf/macros.xacro (robot description, xacro)
@@ -263,6 +263,6 @@
       <inertial>
         <origin xyz="-0.25 0 -0.2" rpy="0 0 0" />
-        <mass value="10"/>
-        <sphere_inertia m="${10}" r="${0.05}"/>
+        <mass value="3"/>
+        <sphere_inertia m="${3}" r="${0.05}"/>
       </inertial>
       <gravity>1</gravity>
@@ -295,6 +295,6 @@
       <inertial>
         <origin xyz="-0.25 -0.2 -0.2" rpy="0 0 0" />
-        <mass value="10"/>
-        <sphere_inertia m="${10}" r="${0.05}"/>
+        <mass value="3"/>
+        <sphere_inertia m="${3}" r="${0.05}"/>
       </inertial>
       <gravity>1</gravity>
@@ -327,6 +327,6 @@
       <inertial>
         <origin xyz="-0.25 0 -0.2" rpy="0 0 0" />
-        <mass value="10"/>
-        <sphere_inertia m="${10}" r="${0.05}"/>
+        <mass value="3"/>
+        <sphere_inertia m="${3}" r="${0.05}"/>
       </inertial>
       <gravity>1</gravity>

Commit message: cool tool 1

File: oz440_description/urdf/macros.xacro (robot description, xacro)
@@ -262,5 +262,5 @@
     <link name="tool1">
       <inertial>
-        <origin xyz="-0.25 0 -0.2" rpy="0 0 0" />
+        <origin xyz="-0.25 0 -0.21" rpy="0 0 0" />
         <mass value="3"/>
         <sphere_inertia m="${3}" r="${0.05}"/>
@@ -268,5 +268,5 @@
       <gravity>1</gravity>
       <collision name="sphere">
-        <origin xyz="-0.25 0 -0.2" rpy="0 0 0"/>
+        <origin xyz="-0.25 0 -0.21" rpy="0 0 0"/>
         <geometry>
           <sphere radius="0.02"/>
@@ -274,5 +274,5 @@
       </collision>
       <visual>
-        <origin xyz="-0.25 0 -0.2" rpy="0 0 0"/>
+        <origin xyz="-0.25 0 -0.21" rpy="0 0 0"/>
         <geometry>
           <sphere radius="0.02"/>
@@ -286,7 +286,7 @@
       </visual>
       <visual>
-        <origin xyz="-0.25 0 -0.165" rpy="0 0 0"/>
-        <geometry>
-          <cylinder radius="0.007" length="0.035"/>
+        <origin xyz="-0.25 0 -0.175" rpy="0 0 0"/>
+        <geometry>
+          <cylinder radius="0.007" length="0.055"/>
         </geometry>
       </visual>
@@ -294,5 +294,5 @@
     <link name="tool2">
       <inertial>
-        <origin xyz="-0.25 -0.2 -0.2" rpy="0 0 0" />
+        <origin xyz="-0.25 -0.2 -0.21" rpy="0 0 0" />
         <mass value="3"/>
         <sphere_inertia m="${3}" r="${0.05}"/>
@@ -300,5 +300,5 @@
       <gravity>1</gravity>
       <collision name="sphere">
-        <origin xyz="-0.25 0 -0.2" rpy="0 0 0"/>
+        <origin xyz="-0.25 0 -0.21" rpy="0 0 0"/>
         <geometry>
           <sphere radius="0.02"/>
@@ -306,5 +306,5 @@
       </collision>
       <visual>
-        <origin xyz="-0.25 0 -0.2" rpy="0 0 0"/>
+        <origin xyz="-0.25 0 -0.21" rpy="0 0 0"/>
         <geometry>
           <sphere radius="0.02"/>
@@ -318,7 +318,7 @@
       </visual>
       <visual>
-        <origin xyz="-0.25 0 -0.165" rpy="0 0 0"/>
-        <geometry>
-          <cylinder radius="0.007" length="0.035"/>
+        <origin xyz="-0.25 0 -0.175" rpy="0 0 0"/>
+        <geometry>
+          <cylinder radius="0.007" length="0.055"/>
         </geometry>
       </visual>
@@ -326,5 +326,5 @@
     <link name="tool3">
       <inertial>
-        <origin xyz="-0.25 0 -0.2" rpy="0 0 0" />
+        <origin xyz="-0.25 0 -0.21" rpy="0 0 0" />
         <mass value="3"/>
         <sphere_inertia m="${3}" r="${0.05}"/>
@@ -332,5 +332,5 @@
       <gravity>1</gravity>
       <collision name="sphere">
-        <origin xyz="-0.25 0 -0.2" rpy="0 0 0"/>
+        <origin xyz="-0.25 0 -0.21" rpy="0 0 0"/>
         <geometry>
           <sphere radius="0.02"/>
@@ -338,5 +338,5 @@
       </collision>
       <visual>
-        <origin xyz="-0.25 0 -0.2" rpy="0 0 0"/>
+        <origin xyz="-0.25 0 -0.21" rpy="0 0 0"/>
         <geometry>
           <sphere radius="0.02"/>
@@ -350,7 +350,7 @@
       </visual>
       <visual>
-        <origin xyz="-0.25 0 -0.165" rpy="0 0 0"/>
-        <geometry>
-          <cylinder radius="0.007" length="0.035"/>
+        <origin xyz="-0.25 0 -0.175" rpy="0 0 0"/>
+        <geometry>
+          <cylinder radius="0.007" length="0.055"/>
         </geometry>
       </visual>

Commit message: cool tool 1

File: oz440_description/urdf/macros.xacro (robot description, xacro)
@@ -60,5 +60,5 @@
       <mu1 value="0.99"/>
       <mu2 value="0.99"/>
-      <kp  value="1e+6" />
+      <kp  value="1e+7" />
       <kd  value="1.0" />
       <material>Gazebo/Black</material>
@@ -69,5 +69,5 @@
       <origin xyz="${tX*wheels_spacing/2} ${tY*((chassis_bottom_width/2)+wheel_chassis_bottom_spacing+(wheel_width/2))} ${wheel_transmission_height-chassis_bottom_height/2}" rpy="0 0 0" />
       <axis xyz="0 1 0" rpy="0 0 0" />
-      <dynamics damping="0.1" friction="0.0"/>
+      <dynamics damping="0.0" friction="0.0"/>
     </joint>
     <transmission name="${fb}_${lr}_trans">
@@ -263,6 +263,6 @@
       <inertial>
         <origin xyz="-0.25 0 -0.21" rpy="0 0 0" />
-        <mass value="3"/>
-        <sphere_inertia m="${3}" r="${0.05}"/>
+        <mass value="0.1"/>
+        <sphere_inertia m="${0.1}" r="${0.05}"/>
       </inertial>
       <gravity>1</gravity>
@@ -295,6 +295,6 @@
       <inertial>
         <origin xyz="-0.25 -0.2 -0.21" rpy="0 0 0" />
-        <mass value="3"/>
-        <sphere_inertia m="${3}" r="${0.05}"/>
+        <mass value="0.1"/>
+        <sphere_inertia m="${0.1}" r="${0.05}"/>
       </inertial>
       <gravity>1</gravity>
@@ -327,6 +327,6 @@
       <inertial>
         <origin xyz="-0.25 0 -0.21" rpy="0 0 0" />
-        <mass value="3"/>
-        <sphere_inertia m="${3}" r="${0.05}"/>
+        <mass value="0.1"/>
+        <sphere_inertia m="${0.1}" r="${0.05}"/>
       </inertial>
       <gravity>1</gravity>

Commit message: cool tool 2

File: oz440_description/urdf/macros.xacro (robot description, xacro)
@@ -24,29 +24,28 @@
     />
   </xacro:macro>
-  <!-- macro pour creer une roue -->
-  <xacro:macro name="wheel" params="fb lr tX tY">
+  <!-- macro pour creer une roue droite  -->
+  <xacro:macro name="right_wheel" params="fb lr tX tY">
     <link name="${fb}_${lr}_wheel">
       <collision>
+        <!--<origin xyz="0 0 0" rpy="0 ${PI/2} ${PI/2}" />-->
+        <origin xyz="${-wheel_diameter/2} ${wheel_width/2} -${wheel_diameter/2}" rpy="0 0 ${-PI/2}" />
+        <geometry>
+          <!--<cylinder length="${wheel_width}" radius="${wheel_diameter/2}"/>-->
+          <mesh filename="model://Wheel/pneu.dae" scale ="0.001 0.001 0.001" />
+        </geometry>
+      </collision>
+      <visual>
         <origin xyz="0 0 0" rpy="0 ${PI/2} ${PI/2}" />
-        <!--<origin xyz="${wheel_diameter/2} -${wheel_width/2} -${wheel_diameter/2}" rpy="0 0 ${PI/2}" />-->
-        <geometry>
-          <cylinder length="${wheel_width}" radius="${wheel_diameter/2}"/>
-          <!--<mesh filename="model://Wheel/pneu.dae" scale ="0.001 0.001 0.001" />-->
-        </geometry>
-      </collision>
-      <!--<visual>-->
+        <geometry>
+          <cylinder length="${wheel_width-0.02}" radius="${wheel_diameter/4}"/>
+        </geometry>
+      </visual>
+      <visual>
         <!--<origin xyz="0 0 0" rpy="0 ${PI/2} ${PI/2}" />-->
-        <!--<geometry>-->
-          <!--<cylinder length="${wheel_width}" radius="${wheel_diameter/4}"/>-->
-        <!--</geometry>-->
-      <!--</visual>-->
-      <visual>
-        <origin xyz="0 0 0" rpy="0 ${PI/2} ${PI/2}" />
-        <!--<origin xyz="${wheel_diameter/2} -${wheel_width/2} -${wheel_diameter/2}" rpy="0 0 ${PI/2}" />-->
-        <geometry>
-          <cylinder length="${wheel_width}" radius="${wheel_diameter/2}"/>
-          <!--<mesh filename="model://Wheel/pneu.dae" scale ="0.001 0.001 0.001" />-->
-        </geometry>
-        <material name="black"/>
+        <origin xyz="${-wheel_diameter/2} ${wheel_width/2} -${wheel_diameter/2}" rpy="0 0 ${-PI/2}" />
+        <geometry>
+          <!--<cylinder length="${wheel_width}" radius="${wheel_diameter/2}"/>-->
+          <mesh filename="model://Wheel/pneu.dae" scale ="0.001 0.001 0.001" />
+        </geometry>
       </visual>
       <inertial>
@@ -60,7 +59,7 @@
       <mu1 value="0.99"/>
       <mu2 value="0.99"/>
-      <kp  value="1e+7" />
-      <kd  value="1.0" />
-      <material>Gazebo/Black</material>
+      <kp  value="1e+6" />
+      <kd  value="1.0" />
+      <material>Gazebo/DarkGrey</material>
     </gazebo>
     <joint name="${fb}_${lr}_wheel_hinge" type="continuous">
@@ -81,4 +80,60 @@
       </actuator>
     </transmission>
+  </xacro:macro><!-- macro pour creer une roue -->
+  <xacro:macro name="left_wheel" params="fb lr tX tY">
+    <link name="${fb}_${lr}_wheel">
+      <collision>
+        <!--<origin xyz="0 0 0" rpy="0 ${PI/2} ${PI/2}" />-->
+        <origin xyz="${wheel_diameter/2} -${wheel_width/2} -${wheel_diameter/2}" rpy="0 0 ${PI/2}" />
+        <geometry>
+          <!--<cylinder length="${wheel_width}" radius="${wheel_diameter/2}"/>-->
+          <mesh filename="model://Wheel/pneu.dae" scale ="0.001 0.001 0.001" />
+        </geometry>
+      </collision>
+      <visual>
+        <origin xyz="0 0 0" rpy="0 ${PI/2} ${PI/2}" />
+        <geometry>
+          <cylinder length="${wheel_width-0.02}" radius="${wheel_diameter/4}"/>
+        </geometry>
+      </visual>
+      <visual>
+        <!--<origin xyz="0 0 0" rpy="0 ${PI/2} ${PI/2}" />-->
+        <origin xyz="${wheel_diameter/2} -${wheel_width/2} -${wheel_diameter/2}" rpy="0 0 ${PI/2}" />
+        <geometry>
+          <!--<cylinder length="${wheel_width}" radius="${wheel_diameter/2}"/>-->
+          <mesh filename="model://Wheel/pneu.dae" scale ="0.001 0.001 0.001" />
+        </geometry>
+      </visual>
+      <inertial>
+        <origin xyz="0 0 0" rpy="0 ${PI/2} ${PI/2}" />
+        <mass value="${wheel_mass}"/>
+        <cylinder_inertia m="${wheel_mass}" r="${wheel_diameter/2}" h="${wheel_width}"/>
+      </inertial>
+    </link>
+    <gazebo reference="${fb}_${lr}_wheel">
+      <gravity>true</gravity>
+      <mu1 value="0.99"/>
+      <mu2 value="0.99"/>
+      <kp  value="1e+6" />
+      <kd  value="1.0" />
+      <material>Gazebo/DarkGrey</material>
+    </gazebo>
+    <joint name="${fb}_${lr}_wheel_hinge" type="continuous">
+      <parent link="chassis_bottom"/>
+      <child link="${fb}_${lr}_wheel"/>
+      <origin xyz="${tX*wheels_spacing/2} ${tY*((chassis_bottom_width/2)+wheel_chassis_bottom_spacing+(wheel_width/2))} ${wheel_transmission_height-chassis_bottom_height/2}" rpy="0 0 0" />
+      <axis xyz="0 1 0" rpy="0 0 0" />
+      <dynamics damping="0.0" friction="0.0"/>
+    </joint>
+    <transmission name="${fb}_${lr}_trans">
+      <type>transmission_interface/SimpleTransmission</type>
+      <joint name="${fb}_${lr}_wheel_hinge">
+        <hardwareInterface>EffortJointInterface</hardwareInterface>
+      </joint>
+      <actuator name="${fb}_${lr}_Motor">
+        <hardwareInterface>EffortJointInterface</hardwareInterface>
+        <mechanicalRedu.ction>46</mechanicalRedu.ction>
+      </actuator>
+    </transmission>
   </xacro:macro>
   <!-- macro pour le porte outils -->
@@ -230,5 +285,5 @@
       <axis rpy="0 0 0" xyz="0 0 1"/>
       <limit upper="0" lower="-0.15" effort="100" velocity="1"/>
-      <dynamics damping="0.7" friction="0.9"/>
+      <dynamics damping="0.9" friction="0.98"/>
     </joint>
     <transmission name="actuator_base_link_to_actuator_part1_trans">
@@ -263,6 +318,6 @@
       <inertial>
         <origin xyz="-0.25 0 -0.21" rpy="0 0 0" />
-        <mass value="0.1"/>
-        <sphere_inertia m="${0.1}" r="${0.05}"/>
+        <mass value="5"/>
+        <sphere_inertia m="${5}" r="${0.04}"/>
       </inertial>
       <gravity>1</gravity>
@@ -270,5 +325,5 @@
         <origin xyz="-0.25 0 -0.21" rpy="0 0 0"/>
         <geometry>
-          <sphere radius="0.02"/>
+          <sphere radius="0.03"/>
         </geometry>
       </collision>
@@ -276,5 +331,5 @@
         <origin xyz="-0.25 0 -0.21" rpy="0 0 0"/>
         <geometry>
-          <sphere radius="0.02"/>
+          <sphere radius="0.03"/>
         </geometry>
       </visual>
@@ -295,6 +350,6 @@
       <inertial>
         <origin xyz="-0.25 -0.2 -0.21" rpy="0 0 0" />
-        <mass value="0.1"/>
-        <sphere_inertia m="${0.1}" r="${0.05}"/>
+        <mass value="5"/>
+        <sphere_inertia m="${5}" r="${0.04}"/>
       </inertial>
       <gravity>1</gravity>
@@ -302,5 +357,5 @@
         <origin xyz="-0.25 0 -0.21" rpy="0 0 0"/>
         <geometry>
-          <sphere radius="0.02"/>
+          <sphere radius="0.03"/>
         </geometry>
       </collision>
@@ -308,5 +363,5 @@
         <origin xyz="-0.25 0 -0.21" rpy="0 0 0"/>
         <geometry>
-          <sphere radius="0.02"/>
+          <sphere radius="0.03"/>
         </geometry>
       </visual>
@@ -327,6 +382,6 @@
       <inertial>
         <origin xyz="-0.25 0 -0.21" rpy="0 0 0" />
-        <mass value="0.1"/>
-        <sphere_inertia m="${0.1}" r="${0.05}"/>
+        <mass value="5"/>
+        <sphere_inertia m="${5}" r="${0.04}"/>
       </inertial>
       <gravity>1</gravity>
@@ -334,5 +389,5 @@
         <origin xyz="-0.25 0 -0.21" rpy="0 0 0"/>
         <geometry>
-          <sphere radius="0.02"/>
+          <sphere radius="0.03"/>
         </geometry>
       </collision>
@@ -340,5 +395,5 @@
         <origin xyz="-0.25 0 -0.21" rpy="0 0 0"/>
         <geometry>
-          <sphere radius="0.02"/>
+          <sphere radius="0.03"/>
         </geometry>
       </visual>
@@ -359,5 +414,5 @@
       <mu1 value="0.99"/>
       <mu2 value="0.99"/>
-      <kp  value="1e+4" />
+      <kp  value="1e+2" />
       <kd  value="1.0" />
       <fdir1 value="0 0 0"/>
@@ -367,5 +422,5 @@
       <mu1 value="0.99"/>
       <mu2 value="0.99"/>
-      <kp  value="1e+4" />
+      <kp  value="1e+2" />
       <kd  value="1.0" />
       <fdir1 value="0 0 0"/>
@@ -375,5 +430,5 @@
       <mu1 value="0.99"/>
       <mu2 value="0.99"/>
-      <kp  value="1e+4" />
+      <kp  value="1e+2" />
       <kd  value="1.0" />
       <fdir1 value="0 0 0"/>
@@ -514,4 +569,31 @@
       <material>Gazebo/Grey</material>
     </gazebo>
+    <link name="IMU_light">
+      <collision>
+        <origin xyz="0 0 0" rpy="0 0 0"/>
+        <geometry>
+          <cylinder radius="0.01" length="0.01"/>
+        </geometry>
+      </collision>
+      <visual>
+        <origin xyz="0 0 0" rpy="0 0 0"/>
+        <geometry>
+          <cylinder radius="0.01" length="0.01"/>
+        </geometry>
+      </visual>
+      <inertial>
+        <mass value="0.1"/>
+        <origin xyz="0 0 0" rpy="0 0 0"/>
+        <sphere_inertia m="0.1" r="0.01"/>
+      </inertial>
+    </link>
+    <gazebo reference="IMU_light">
+      <mu1 value="0.99"/>
+      <mu2 value="0.99"/>
+      <kp  value="1e+7" />
+      <kd  value="1.0" />
+      <fdir1 value="0 0 0"/>
+      <material>Gazebo/Red</material>
+    </gazebo>
     <joint name="actuator_base_to_IMU_base_joint" type="fixed">
       <parent link="${parent}"/>
@@ -524,4 +606,9 @@
       <origin xyz="${IMU_base_Length/2-IMU_Length/2} 0 ${IMU_base_Height/2+IMU_Height/2}" rpy="0 0 0"/>
     </joint>
+    <joint name="IMU_to_IMU_light" type="fixed">
+      <parent link="IMU_link"/>
+      <child link="IMU_light"/>
+      <origin xyz="0 -0.03 ${IMU_Height/2+0.005}" rpy="0 0 0"/>
+    </joint>
   </xacro:macro>
   <!-- macro pour le bumper -->

File: oz440_description/urdf/oz440.xacro (robot description, xacro)
@@ -65,8 +65,8 @@
 	<tool_macro parent="actuator_part2_link"/>
     <!-- inclusion des roues -->
-	<wheel fb="front" lr="right" tX="1" tY="-1"/>
-	<wheel fb="front" lr="left" tX="1" tY="1"/>
-	<wheel fb="back" lr="right" tX="-1" tY="-1"/>
-	<wheel fb="back" lr="left" tX="-1" tY="1"/>
+	<right_wheel fb="front" lr="right" tX="1" tY="-1"/>
+	<left_wheel fb="front" lr="left" tX="1" tY="1"/>
+	<right_wheel fb="back" lr="right" tX="-1" tY="-1"/>
+	<left_wheel fb="back" lr="left" tX="-1" tY="1"/>
 	<!-- inclusion de la camera stereo -->
 	<camera_stereo parent="chassis_bottom"/>

File: oz440_description/urdf/properties.xacro (robot description, xacro)
@@ -5,5 +5,5 @@
 	<!-- Proprietes de la partie basse du robot -->
 	<xacro:property name="chassis_bottom_height" value="0.243"/>
-	<xacro:property name="chassis_bottom_width" value="0.17340"/>
+	<xacro:property name="chassis_bottom_width" value="0.20"/>
 	<xacro:property name="chassis_bottom_length" value="0.67454"/>
 	<xacro:property name="chassis_bottom_mass" value="30"/>
@@ -14,8 +14,9 @@
 	<xacro:property name="chassis_top_mass" value="70"/>
 	<!-- Proprietes des roues -->
-	<xacro:property name="wheel_diameter" value="0.292"/>
-	<xacro:property name="wheel_width" value="0.08786"/>
+	<!--<xacro:property name="wheel_diameter" value="0.292"/>-->
+	<xacro:property name="wheel_diameter" value="0.3092"/>
+	<xacro:property name="wheel_width" value="0.08761"/>
 	<xacro:property name="wheel_transmission_height" value="0.058"/>
-	<xacro:property name="wheel_chassis_bottom_spacing" value="0.03430"/>
+	<xacro:property name="wheel_chassis_bottom_spacing" value="0.01"/>
 	<xacro:property name="wheels_spacing" value="0.435"/>
 	<xacro:property name="wheel_mass" value="3"/>
@@ -25,5 +26,5 @@
 	<xacro:property name="actuator_base_Width" value="0.1"/>
 	<xacro:property name="actuator_base_Height" value="0.2"/>
-	<xacro:property name="actuator_base_chassis_spacing" value="0.02"/>
+	<xacro:property name="actuator_base_chassis_spacing" value="0.01"/>
 	<xacro:property name="actuator_part1_Mass" value="1"/>
 	<xacro:property name="actuator_part1_Length" value="0.05"/>
@@ -31,6 +32,6 @@
 	<xacro:property name="actuator_part1_Height" value="0.05"/>
 	<xacro:property name="actuator_part2_Mass" value="1"/>
-	<xacro:property name="actuator_part2_Length" value="0.04"/>
-	<xacro:property name="actuator_part2_Width" value="0.04"/>
+	<xacro:property name="actuator_part2_Length" value="0.035"/>
+	<xacro:property name="actuator_part2_Width" value="0.035"/>
 	<xacro:property name="actuator_part2_Height" value="0.04"/>
 	<!-- Proprietes de la camera -->
@@ -54,7 +55,7 @@
 	<xacro:property name="IMU_base_Height" value="0.1"/>
 	<xacro:property name="IMU_Mass" value="0.2"/>
-	<xacro:property name="IMU_Length" value="0.1"/>
+	<xacro:property name="IMU_Length" value="0.05"/>
 	<xacro:property name="IMU_Width" value="0.1"/>
-	<xacro:property name="IMU_Height" value="0.06"/>
+	<xacro:property name="IMU_Height" value="0.05"/>
 	<!-- Proprietes du bumper -->
 	<xacro:property name="bumper_base_Mass" value="0.3"/>

Commit message: friction = 1 tool

File: oz440_description/urdf/macros.xacro (robot description, xacro)
@@ -285,5 +285,5 @@
       <axis rpy="0 0 0" xyz="0 0 1"/>
       <limit upper="0" lower="-0.15" effort="100" velocity="1"/>
-      <dynamics damping="0.9" friction="0.98"/>
+      <dynamics damping="0.7" friction="1.0"/>
     </joint>
     <transmission name="actuator_base_link_to_actuator_part1_trans">

Commit message: friction = 1 tool

File: oz440_description/urdf/macros.xacro (robot description, xacro)
@@ -59,5 +59,5 @@
       <mu1 value="0.99"/>
       <mu2 value="0.99"/>
-      <kp  value="5000000" />
+      <kp  value="1000000" />
       <kd  value="1.0" />
       <material>Gazebo/DarkGrey</material>
@@ -115,5 +115,5 @@
       <mu1 value="0.99"/>
       <mu2 value="0.99"/>
-      <kp  value="5000000" />
+      <kp  value="1000000" />
       <kd  value="1.0" />
       <material>Gazebo/DarkGrey</material>
@@ -285,5 +285,5 @@
       <axis rpy="0 0 0" xyz="0 0 1"/>
       <limit upper="0" lower="-0.15" effort="100" velocity="1"/>
-      <dynamics damping="0.7" friction="1.0"/>
+      <dynamics damping="0.7" friction="0.98"/>
     </joint>
     <transmission name="actuator_base_link_to_actuator_part1_trans">
@@ -318,6 +318,6 @@
       <inertial>
         <origin xyz="-0.25 0 -0.21" rpy="0 0 0" />
-        <mass value="5"/>
-        <sphere_inertia m="${5}" r="${0.04}"/>
+        <mass value="2"/>
+        <sphere_inertia m="${2}" r="${0.04}"/>
       </inertial>
       <gravity>1</gravity>
@@ -350,6 +350,6 @@
       <inertial>
         <origin xyz="-0.25 -0.2 -0.21" rpy="0 0 0" />
-        <mass value="5"/>
-        <sphere_inertia m="${5}" r="${0.04}"/>
+        <mass value="2"/>
+        <sphere_inertia m="${2}" r="${0.04}"/>
       </inertial>
       <gravity>1</gravity>
@@ -382,6 +382,6 @@
       <inertial>
         <origin xyz="-0.25 0 -0.21" rpy="0 0 0" />
-        <mass value="5"/>
-        <sphere_inertia m="${5}" r="${0.04}"/>
+        <mass value="2"/>
+        <sphere_inertia m="${2}" r="${0.04}"/>
       </inertial>
       <gravity>1</gravity>

File: oz440_description/urdf/properties.xacro (robot description, xacro)
@@ -27,9 +27,9 @@
 	<xacro:property name="actuator_base_Height" value="0.2"/>
 	<xacro:property name="actuator_base_chassis_spacing" value="0.01"/>
-	<xacro:property name="actuator_part1_Mass" value="1"/>
+	<xacro:property name="actuator_part1_Mass" value="0.5"/>
 	<xacro:property name="actuator_part1_Length" value="0.05"/>
 	<xacro:property name="actuator_part1_Width" value="0.41"/>
 	<xacro:property name="actuator_part1_Height" value="0.05"/>
-	<xacro:property name="actuator_part2_Mass" value="1"/>
+	<xacro:property name="actuator_part2_Mass" value="0.5"/>
 	<xacro:property name="actuator_part2_Length" value="0.035"/>
 	<xacro:property name="actuator_part2_Width" value="0.035"/>

Commit message: old wheel collision

File: oz440_description/urdf/macros.xacro (robot description, xacro)
@@ -28,9 +28,9 @@
     <link name="${fb}_${lr}_wheel">
       <collision>
-        <!--<origin xyz="0 0 0" rpy="0 ${PI/2} ${PI/2}" />-->
-        <origin xyz="${-wheel_diameter/2} ${wheel_width/2} -${wheel_diameter/2}" rpy="0 0 ${-PI/2}" />
-        <geometry>
-          <!--<cylinder length="${wheel_width}" radius="${wheel_diameter/2}"/>-->
-          <mesh filename="model://Wheel/pneu.dae" scale ="0.001 0.001 0.001" />
+        <origin xyz="0 0 0" rpy="0 ${PI/2} ${PI/2}" />
+        <!--<origin xyz="${-wheel_diameter/2} ${wheel_width/2} -${wheel_diameter/2}" rpy="0 0 ${-PI/2}" />-->
+        <geometry>
+          <cylinder length="${wheel_width}" radius="${wheel_diameter/2}"/>
+          <!--<mesh filename="model://Wheel/pneu.dae" scale ="0.001 0.001 0.001" />-->
         </geometry>
       </collision>
