Commit message: old wheel collision

File: oz440_description/urdf/macros.xacro (robot description, xacro)
@@ -59,5 +59,5 @@
       <mu1 value="0.99"/>
       <mu2 value="0.99"/>
-      <kp  value="1000000" />
+      <kp  value="1e+7" />
       <kd  value="1.0" />
       <material>Gazebo/DarkGrey</material>
@@ -84,9 +84,9 @@
     <link name="${fb}_${lr}_wheel">
       <collision>
-        <!--<origin xyz="0 0 0" rpy="0 ${PI/2} ${PI/2}" />-->
-        <origin xyz="${wheel_diameter/2} -${wheel_width/2} -${wheel_diameter/2}" rpy="0 0 ${PI/2}" />
-        <geometry>
-          <!--<cylinder length="${wheel_width}" radius="${wheel_diameter/2}"/>-->
-          <mesh filename="model://Wheel/pneu.dae" scale ="0.001 0.001 0.001" />
+        <origin xyz="0 0 0" rpy="0 ${PI/2} ${PI/2}" />
+        <!--<origin xyz="${wheel_diameter/2} -${wheel_width/2} -${wheel_diameter/2}" rpy="0 0 ${PI/2}" />-->
+        <geometry>
+          <cylinder length="${wheel_width}" radius="${wheel_diameter/2}"/>
+          <!--<mesh filename="model://Wheel/pneu.dae" scale ="0.001 0.001 0.001" />-->
         </geometry>
       </collision>
@@ -115,5 +115,5 @@
       <mu1 value="0.99"/>
       <mu2 value="0.99"/>
-      <kp  value="1000000" />
+      <kp  value="1e+7" />
       <kd  value="1.0" />
       <material>Gazebo/DarkGrey</material>

Commit message: old wheel collision

File: oz440_description/urdf/macros.xacro (robot description, xacro)
@@ -318,6 +318,6 @@
       <inertial>
         <origin xyz="-0.25 0 -0.21" rpy="0 0 0" />
-        <mass value="2"/>
-        <sphere_inertia m="${2}" r="${0.04}"/>
+        <mass value="4"/>
+        <sphere_inertia m="${4}" r="${0.04}"/>
       </inertial>
       <gravity>1</gravity>
@@ -350,6 +350,6 @@
       <inertial>
         <origin xyz="-0.25 -0.2 -0.21" rpy="0 0 0" />
-        <mass value="2"/>
-        <sphere_inertia m="${2}" r="${0.04}"/>
+        <mass value="4"/>
+        <sphere_inertia m="${4}" r="${0.04}"/>
       </inertial>
       <gravity>1</gravity>
@@ -382,6 +382,6 @@
       <inertial>
         <origin xyz="-0.25 0 -0.21" rpy="0 0 0" />
-        <mass value="2"/>
-        <sphere_inertia m="${2}" r="${0.04}"/>
+        <mass value="4"/>
+        <sphere_inertia m="${4}" r="${0.04}"/>
       </inertial>
       <gravity>1</gravity>
@@ -414,5 +414,5 @@
       <mu1 value="0.99"/>
       <mu2 value="0.99"/>
-      <kp  value="1e+2" />
+      <kp  value="1e+6" />
       <kd  value="1.0" />
       <fdir1 value="0 0 0"/>
@@ -422,5 +422,5 @@
       <mu1 value="0.99"/>
       <mu2 value="0.99"/>
-      <kp  value="1e+2" />
+      <kp  value="1e+6" />
       <kd  value="1.0" />
       <fdir1 value="0 0 0"/>
@@ -430,5 +430,5 @@
       <mu1 value="0.99"/>
       <mu2 value="0.99"/>
-      <kp  value="1e+2" />
+      <kp  value="1e+6" />
       <kd  value="1.0" />
       <fdir1 value="0 0 0"/>

Commit message: old wheel collision

File: oz440_description/urdf/macros.xacro (robot description, xacro)
@@ -3,663 +3,630 @@
 Les proprietes sont modifiables dans le fichiers properties.xacro -->
 <robot name="oz440" xmlns:xacro="http://www.ros.org/wiki/xacro">
-  <!-- macro pour calculer l'inertie d'un cylindre -->
-  <xacro:macro name="cylinder_inertia" params="m r h">
-    <inertia  ixx="${m*(3*r*r+h*h)/12}" ixy = "0" ixz = "0"
-              iyy="${m*(3*r*r+h*h)/12}" iyz = "0"
-              izz="${m*r*r/2}"
-    />
-  </xacro:macro>
-  <!-- macro pour calculer l'inertie d'un pave -->
-  <xacro:macro name="box_inertia" params="m x y z">
-    <inertia  ixx="${m*(y*y+z*z)/12}" ixy = "0" ixz = "0"
-              iyy="${m*(x*x+z*z)/12}" iyz = "0"
-              izz="${m*(x*x+z*z)/12}"
-    />
-  </xacro:macro>
-  <!-- macro pour calculer l'inertie d'une sphere -->
-  <xacro:macro name="sphere_inertia" params="m r">
-    <inertia  ixx="${2*m*r*r/5}" ixy = "0" ixz = "0"
-              iyy="${2*m*r*r/5}" iyz = "0"
-              izz="${2*m*r*r/5}"
-    />
-  </xacro:macro>
-  <!-- macro pour creer une roue droite  -->
-  <xacro:macro name="right_wheel" params="fb lr tX tY">
-    <link name="${fb}_${lr}_wheel">
-      <collision>
-        <origin xyz="0 0 0" rpy="0 ${PI/2} ${PI/2}" />
-        <!--<origin xyz="${-wheel_diameter/2} ${wheel_width/2} -${wheel_diameter/2}" rpy="0 0 ${-PI/2}" />-->
-        <geometry>
-          <cylinder length="${wheel_width}" radius="${wheel_diameter/2}"/>
-          <!--<mesh filename="model://Wheel/pneu.dae" scale ="0.001 0.001 0.001" />-->
-        </geometry>
-      </collision>
-      <visual>
-        <origin xyz="0 0 0" rpy="0 ${PI/2} ${PI/2}" />
-        <geometry>
-          <cylinder length="${wheel_width-0.02}" radius="${wheel_diameter/4}"/>
-        </geometry>
-      </visual>
-      <visual>
-        <!--<origin xyz="0 0 0" rpy="0 ${PI/2} ${PI/2}" />-->
-        <origin xyz="${-wheel_diameter/2} ${wheel_width/2} -${wheel_diameter/2}" rpy="0 0 ${-PI/2}" />
-        <geometry>
-          <!--<cylinder length="${wheel_width}" radius="${wheel_diameter/2}"/>-->
-          <mesh filename="model://Wheel/pneu.dae" scale ="0.001 0.001 0.001" />
-        </geometry>
-      </visual>
-      <inertial>
-        <origin xyz="0 0 0" rpy="0 ${PI/2} ${PI/2}" />
-        <mass value="${wheel_mass}"/>
-        <cylinder_inertia m="${wheel_mass}" r="${wheel_diameter/2}" h="${wheel_width}"/>
-      </inertial>
-    </link>
-    <gazebo reference="${fb}_${lr}_wheel">
-      <gravity>true</gravity>
-      <mu1 value="0.99"/>
-      <mu2 value="0.99"/>
-      <kp  value="1e+7" />
-      <kd  value="1.0" />
-      <material>Gazebo/DarkGrey</material>
-    </gazebo>
-    <joint name="${fb}_${lr}_wheel_hinge" type="continuous">
-      <parent link="chassis_bottom"/>
-      <child link="${fb}_${lr}_wheel"/>
-      <origin xyz="${tX*wheels_spacing/2} ${tY*((chassis_bottom_width/2)+wheel_chassis_bottom_spacing+(wheel_width/2))} ${wheel_transmission_height-chassis_bottom_height/2}" rpy="0 0 0" />
-      <axis xyz="0 1 0" rpy="0 0 0" />
-      <dynamics damping="0.0" friction="0.0"/>
-    </joint>
-    <transmission name="${fb}_${lr}_trans">
-      <type>transmission_interface/SimpleTransmission</type>
-      <joint name="${fb}_${lr}_wheel_hinge">
-        <hardwareInterface>EffortJointInterface</hardwareInterface>
-      </joint>
-      <actuator name="${fb}_${lr}_Motor">
-        <hardwareInterface>EffortJointInterface</hardwareInterface>
-        <mechanicalRedu.ction>46</mechanicalRedu.ction>
-      </actuator>
-    </transmission>
-  </xacro:macro><!-- macro pour creer une roue -->
-  <xacro:macro name="left_wheel" params="fb lr tX tY">
-    <link name="${fb}_${lr}_wheel">
-      <collision>
-        <origin xyz="0 0 0" rpy="0 ${PI/2} ${PI/2}" />
-        <!--<origin xyz="${wheel_diameter/2} -${wheel_width/2} -${wheel_diameter/2}" rpy="0 0 ${PI/2}" />-->
-        <geometry>
-          <cylinder length="${wheel_width}" radius="${wheel_diameter/2}"/>
-          <!--<mesh filename="model://Wheel/pneu.dae" scale ="0.001 0.001 0.001" />-->
-        </geometry>
-      </collision>
-      <visual>
-        <origin xyz="0 0 0" rpy="0 ${PI/2} ${PI/2}" />
-        <geometry>
-          <cylinder length="${wheel_width-0.02}" radius="${wheel_diameter/4}"/>
-        </geometry>
-      </visual>
-      <visual>
-        <!--<origin xyz="0 0 0" rpy="0 ${PI/2} ${PI/2}" />-->
-        <origin xyz="${wheel_diameter/2} -${wheel_width/2} -${wheel_diameter/2}" rpy="0 0 ${PI/2}" />
-        <geometry>
-          <!--<cylinder length="${wheel_width}" radius="${wheel_diameter/2}"/>-->
-          <mesh filename="model://Wheel/pneu.dae" scale ="0.001 0.001 0.001" />
-        </geometry>
-      </visual>
-      <inertial>
-        <origin xyz="0 0 0" rpy="0 ${PI/2} ${PI/2}" />
-        <mass value="${wheel_mass}"/>
-        <cylinder_inertia m="${wheel_mass}" r="${wheel_diameter/2}" h="${wheel_width}"/>
-      </inertial>
-    </link>
-    <gazebo reference="${fb}_${lr}_wheel">
-      <gravity>true</gravity>
-      <mu1 value="0.99"/>
-      <mu2 value="0.99"/>
-      <kp  value="1e+7" />
-      <kd  value="1.0" />
-      <material>Gazebo/DarkGrey</material>
-    </gazebo>
-    <joint name="${fb}_${lr}_wheel_hinge" type="continuous">
-      <parent link="chassis_bottom"/>
-      <child link="${fb}_${lr}_wheel"/>
-      <origin xyz="${tX*wheels_spacing/2} ${tY*((chassis_bottom_width/2)+wheel_chassis_bottom_spacing+(wheel_width/2))} ${wheel_transmission_height-chassis_bottom_height/2}" rpy="0 0 0" />
-      <axis xyz="0 1 0" rpy="0 0 0" />
-      <dynamics damping="0.0" friction="0.0"/>
-    </joint>
-    <transmission name="${fb}_${lr}_trans">
-      <type>transmission_interface/SimpleTransmission</type>
-      <joint name="${fb}_${lr}_wheel_hinge">
-        <hardwareInterface>EffortJointInterface</hardwareInterface>
-      </joint>
-      <actuator name="${fb}_${lr}_Motor">
-        <hardwareInterface>EffortJointInterface</hardwareInterface>
-        <mechanicalRedu.ction>46</mechanicalRedu.ction>
-      </actuator>
-    </transmission>
-  </xacro:macro>
-  <!-- macro pour le porte outils -->
-  <xacro:macro name="actuator_macro" params="parent">
-    <link name="actuator_base_link">
-      <inertial>
-        <mass value="1"/>
+    <!-- macro pour calculer l'inertie d'un cylindre -->
+    <xacro:macro name="cylinder_inertia" params="m r h">
+        <inertia  ixx="${m*(3*r*r+h*h)/12}" ixy = "0" ixz = "0"
+                  iyy="${m*(3*r*r+h*h)/12}" iyz = "0"
+                  izz="${m*r*r/2}"
+        />
+    </xacro:macro>
+    <!-- macro pour calculer l'inertie d'un pave -->
+    <xacro:macro name="box_inertia" params="m x y z">
+        <inertia  ixx="${m*(y*y+z*z)/12}" ixy = "0" ixz = "0"
+                  iyy="${m*(x*x+z*z)/12}" iyz = "0"
+                  izz="${m*(x*x+z*z)/12}"
+        />
+    </xacro:macro>
+    <!-- macro pour calculer l'inertie d'une sphere -->
+    <xacro:macro name="sphere_inertia" params="m r">
+        <inertia  ixx="${2*m*r*r/5}" ixy = "0" ixz = "0"
+                  iyy="${2*m*r*r/5}" iyz = "0"
+                  izz="${2*m*r*r/5}"
+        />
+    </xacro:macro>
+    <!-- macro pour creer les centres  -->
+    <xacro:macro name="center" params="fb lr tX tY">
+        <link name="${fb}_${lr}_center">
+            <visual>
+                <origin xyz="0 0 0" rpy="0 ${PI/2} ${PI/2}" />
+                <geometry>
+                    <cylinder length="${wheel_width-0.02}" radius="${wheel_diameter/4}"/>
+                </geometry>
+            </visual>
+            <inertial>
+                <origin xyz="0 0 0" rpy="0 ${PI/2} ${PI/2}" />
+                <mass value="${wheel_mass/2}"/>
+                <cylinder_inertia m="${wheel_mass/2}" r="${wheel_diameter/4}" h="${wheel_width}"/>
+            </inertial>
+        </link>
+        <gazebo reference="${fb}_${lr}_center">
+            <gravity>true</gravity>
+            <mu1 value="0.99"/>
+            <mu2 value="0.99"/>
+            <kp  value="1e+7" />
+            <kd  value="1.0" />
+            <material>Gazebo/Grey</material>
+        </gazebo>
+        <joint name="${fb}_${lr}_wheel_to_wheel_center" type="fixed">
+        <parent link="${fb}_${lr}_wheel"/>
+        <child link="${fb}_${lr}_center"/>
         <origin xyz="0 0 0" rpy="0 0 0"/>
-        <box_inertia m="${actuator_base_Mass}" x="${actuator_base_Length}" y="${actuator_base_Width}" z="${actuator_base_Height}"/>
-      </inertial>
-      <collision name="collision_actuator">
-        <origin xyz="0 0 0" rpy="0 0 0"/>
-        <geometry>
-          <box size="${actuator_base_Length} ${actuator_base_Width} ${actuator_base_Height}"/>
-        </geometry>
-      </collision>
-      <visual>
-        <origin xyz="0 0 0" rpy="0 0 0"/>
-        <geometry>
-          <box size="${actuator_base_Length} ${actuator_base_Width} ${actuator_base_Height}"/>
-        </geometry>
-      </visual>
-    </link>
-    <gazebo reference="actuator_base_link">
-      <mu1 value="0.99"/>
-      <mu2 value="0.99"/>
-      <kp  value="1e+7" />
-      <kd  value="1.0" />
-      <fdir1 value="0 0 0"/>
-      <material> Gazebo/white </material>
-    </gazebo>
-    <link name="actuator_part1_link">
-      <inertial>
-        <mass value="${actuator_part1_Mass}"/>
-        <origin xyz="0 0 0" rpy="0 0 0"/>
-        <box_inertia m="${actuator_part1_Mass}" x="${actuator_part1_Length}" y="${actuator_part1_Width}" z="${actuator_part1_Height}"/>
-      </inertial>
-      <collision name="collision_actuator">
-        <origin xyz="0 0 0" rpy="0 0 0"/>
-        <geometry>
-          <box size="${actuator_part1_Length} ${actuator_part1_Width} ${actuator_part1_Height}"/>
-        </geometry>
-      </collision>
-      <visual>
-        <origin xyz="0 0 0" rpy="0 0 0"/>
-        <geometry>
-          <box size="${actuator_part1_Length} ${actuator_part1_Width} ${actuator_part1_Height}"/>
-        </geometry>
-      </visual>
-    </link>
-    <gazebo reference="actuator_part1_link">
-      <mu1 value="0.99"/>
-      <mu2 value="0.99"/>
-      <kp  value="1e+7" />
-      <kd  value="1.0" />
-      <fdir1 value="0 0 0"/>
-      <material>Gazebo/Green</material>
-    </gazebo>
-    <link name="actuator_part21_link">
-      <inertial>
-        <mass value="${actuator_part2_Mass}"/>
-        <origin xyz="0 0 0" rpy="0 0 0"/>
-        <box_inertia m="${actuator_part2_Mass}" x="${actuator_part2_Length}" y="${actuator_part2_Width}" z="${actuator_part2_Height}"/>
-      </inertial>
-      <collision name="collision_actuator">
-        <origin xyz="0 0 0" rpy="0 0 0"/>
-        <geometry>
-          <box size="${actuator_part2_Length} ${actuator_part2_Width} ${actuator_part2_Height}"/>
-        </geometry>
-      </collision>
-      <visual>
-        <origin xyz="0 0 0" rpy="0 0 0"/>
-        <geometry>
-          <box size="${actuator_part2_Length} ${actuator_part2_Width} ${actuator_part2_Height}"/>
-        </geometry>
-      </visual>
-    </link>
-    <link name="actuator_part22_link">
-      <inertial>
-        <mass value="${actuator_part2_Mass}"/>
-        <origin xyz="0 0 0" rpy="0 0 0"/>
-        <box_inertia m="${actuator_part2_Mass}" x="${actuator_part2_Length}" y="${actuator_part2_Width}" z="${actuator_part2_Height}"/>
-      </inertial>
-      <collision name="collision_actuator">
-        <origin xyz="0 0 0" rpy="0 0 0"/>
-        <geometry>
-          <box size="${actuator_part2_Length} ${actuator_part2_Width} ${actuator_part2_Height}"/>
-        </geometry>
-      </collision>
-      <visual>
-        <origin xyz="0 0 0" rpy="0 0 0"/>
-        <geometry>
-          <box size="${actuator_part2_Length} ${actuator_part2_Width} ${actuator_part2_Height}"/>
-        </geometry>
-      </visual>
-    </link>
-    <link name="actuator_part23_link">
-      <inertial>
-        <mass value="${actuator_part2_Mass}"/>
-        <origin xyz="0 0 0" rpy="0 0 0"/>
-        <box_inertia m="${actuator_part2_Mass}" x="${actuator_part2_Length}" y="${actuator_part2_Width}" z="${actuator_part2_Height}"/>
-      </inertial>
-      <collision name="collision_actuator">
-        <origin xyz="0 0 0" rpy="0 0 0"/>
-        <geometry>
-          <box size="${actuator_part2_Length} ${actuator_part2_Width} ${actuator_part2_Height}"/>
-        </geometry>
-      </collision>
-      <visual>
-        <origin xyz="0 0 0" rpy="0 0 0"/>
-        <geometry>
-          <box size="${actuator_part2_Length} ${actuator_part2_Width} ${actuator_part2_Height}"/>
-        </geometry>
-      </visual>
-    </link>
-    <gazebo reference="actuator_part21_link">
-      <mu1 value="0.99"/>
-      <mu2 value="0.99"/>
-      <kp  value="1e+7" />
-      <kd  value="1.0" />
-      <fdir1 value="0 0 0"/>
-      <material>Gazebo/Green</material>
-    </gazebo>
-    <gazebo reference="actuator_part22_link">
-      <mu1 value="0.99"/>
-      <mu2 value="0.99"/>
-      <kp  value="1e+7" />
-      <kd  value="1.0" />
-      <fdir1 value="0 0 0"/>
-      <material>Gazebo/Green</material>
-    </gazebo>
-    <gazebo reference="actuator_part23_link">
-      <mu1 value="0.99"/>
-      <mu2 value="0.99"/>
-      <kp  value="1e+7" />
-      <kd  value="1.0" />
-      <fdir1 value="0 0 0"/>
-      <material>Gazebo/Green</material>
-    </gazebo>
-    <joint name="chassis_bottom_to_actuator_base_joint" type="fixed">
-      <parent link="${parent}"/>
-      <child link="actuator_base_link"/>
-      <origin xyz="${-chassis_bottom_length/2-actuator_base_Length/2-actuator_base_chassis_spacing} 0 ${chassis_bottom_height/2}" rpy="0 0 0"/>
-    </joint>
-    <joint name="actuator_base_link_to_actuator_part1_joint" type="prismatic">
-      <parent link="actuator_base_link"/>
-      <child link="actuator_part1_link"/>
-      <origin xyz="${-actuator_base_Length/2-actuator_part1_Length/2} 0 ${actuator_base_Height/2}" rpy="0 0 0"/>
-      <axis rpy="0 0 0" xyz="0 0 1"/>
-      <limit upper="0" lower="-0.15" effort="100" velocity="1"/>
-      <dynamics damping="0.7" friction="0.98"/>
-    </joint>
-    <transmission name="actuator_base_link_to_actuator_part1_trans">
-      <type>transmission_interface/SimpleTransmission</type>
-      <joint name="actuator_base_link_to_actuator_part1_joint">
-        <hardwareInterface>EffortJointInterface</hardwareInterface>
-      </joint>
-      <actuator name="actuator_base_link_to_actuator_part1_motor">
-        <hardwareInterface>EffortJointInterface</hardwareInterface>
-        <mechanicalRedu.ction>46</mechanicalRedu.ction>
-      </actuator>
-    </transmission>
-    <joint name="actuator_part1_to_actuator_part21_joint" type="fixed">
-      <parent link="actuator_part1_link"/>
-      <child link="actuator_part21_link"/>
-      <origin xyz="0 0 ${-actuator_part1_Height/2-actuator_part2_Height/2}" rpy="0 0 0"/>
-    </joint>
-    <joint name="actuator_part1_to_actuator_part22_joint" type="fixed">
-      <parent link="actuator_part1_link"/>
-      <child link="actuator_part22_link"/>
-      <origin xyz="0 -0.18 ${-actuator_part1_Height/2-actuator_part2_Height/2}" rpy="0 0 0"/>
-    </joint>
-    <joint name="actuator_part1_to_actuator_part23_joint" type="fixed">
-      <parent link="actuator_part1_link"/>
-      <child link="actuator_part23_link"/>
-      <origin xyz="0 0.18 ${-actuator_part1_Height/2-actuator_part2_Height/2}" rpy="0 0 0"/>
-    </joint>
-  </xacro:macro>
-  <!-- macro pour l'outils -->
-  <xacro:macro name="tool_macro" params="parent">
-    <link name="tool1">
-      <inertial>
-        <origin xyz="-0.25 0 -0.21" rpy="0 0 0" />
-        <mass value="4"/>
-        <sphere_inertia m="${4}" r="${0.04}"/>
-      </inertial>
-      <gravity>1</gravity>
-      <collision name="sphere">
-        <origin xyz="-0.25 0 -0.21" rpy="0 0 0"/>
-        <geometry>
-          <sphere radius="0.03"/>
-        </geometry>
-      </collision>
-      <visual>
-        <origin xyz="-0.25 0 -0.21" rpy="0 0 0"/>
-        <geometry>
-          <sphere radius="0.03"/>
-        </geometry>
-      </visual>
-      <visual>
-        <origin xyz="-0.125 0 -0.075" rpy="0 1.03 0"/>
-        <geometry>
-          <cylinder radius="0.007" length="0.29"/>
-        </geometry>
-      </visual>
-      <visual>
-        <origin xyz="-0.25 0 -0.175" rpy="0 0 0"/>
-        <geometry>
-          <cylinder radius="0.007" length="0.055"/>
-        </geometry>
-      </visual>
-    </link>
-    <link name="tool2">
-      <inertial>
-        <origin xyz="-0.25 -0.2 -0.21" rpy="0 0 0" />
-        <mass value="4"/>
-        <sphere_inertia m="${4}" r="${0.04}"/>
-      </inertial>
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
File: oz440_description/urdf/oz440.xacro (robot description, xacro)
@@ -65,8 +65,13 @@
 	<tool_macro parent="actuator_part2_link"/>
     <!-- inclusion des roues -->
-	<right_wheel fb="front" lr="right" tX="1" tY="-1"/>
-	<left_wheel fb="front" lr="left" tX="1" tY="1"/>
-	<right_wheel fb="back" lr="right" tX="-1" tY="-1"/>
-	<left_wheel fb="back" lr="left" tX="-1" tY="1"/>
+	<wheel fb="front" lr="right" tX="1" tY="-1"/>
+	<wheel fb="front" lr="left" tX="1" tY="1"/>
+	<wheel fb="back" lr="right" tX="-1" tY="-1"/>
+	<wheel fb="back" lr="left" tX="-1" tY="1"/>
+	<!-- inclusion des roues -->
+	<center fb="front" lr="right" tX="1" tY="-1"/>
+	<center fb="front" lr="left" tX="1" tY="1"/>
+	<center fb="back" lr="right" tX="-1" tY="-1"/>
+	<center fb="back" lr="left" tX="-1" tY="1"/>
 	<!-- inclusion de la camera stereo -->
 	<camera_stereo parent="chassis_bottom"/>
