Commit message: position

File: oz440_description/urdf/macros.xacro (robot description, xacro)
@@ -284,5 +284,5 @@
         <link name="tool1">
             <inertial>
-                <origin xyz="-0.25 0 -0.21" rpy="0 0 0" />
+                <origin xyz="-0.25 0 -0.22" rpy="0 0 0" />
                 <mass value="4"/>
                 <sphere_inertia m="${4}" r="${0.04}"/>
@@ -290,5 +290,5 @@
             <gravity>1</gravity>
             <collision name="sphere">
-                <origin xyz="-0.25 0 -0.21" rpy="0 0 0"/>
+                <origin xyz="-0.25 0 -0.22" rpy="0 0 0"/>
                 <geometry>
                     <sphere radius="0.03"/>
@@ -296,5 +296,5 @@
             </collision>
             <visual>
-                <origin xyz="-0.25 0 -0.21" rpy="0 0 0"/>
+                <origin xyz="-0.25 0 -0.22" rpy="0 0 0"/>
                 <geometry>
                     <sphere radius="0.03"/>
@@ -304,11 +304,11 @@
                 <origin xyz="-0.125 0 -0.075" rpy="0 1.03 0"/>
                 <geometry>
-                    <cylinder radius="0.007" length="0.29"/>
-                </geometry>
-            </visual>
-            <visual>
-                <origin xyz="-0.25 0 -0.175" rpy="0 0 0"/>
-                <geometry>
-                    <cylinder radius="0.007" length="0.055"/>
+                    <cylinder radius="0.007" length="0.30"/>
+                </geometry>
+            </visual>
+            <visual>
+                <origin xyz="-0.25 0 -0.18" rpy="0 0 0"/>
+                <geometry>
+                    <cylinder radius="0.007" length="0.065"/>
                 </geometry>
             </visual>
@@ -316,5 +316,5 @@
         <link name="tool2">
             <inertial>
-                <origin xyz="-0.25 -0.2 -0.21" rpy="0 0 0" />
+                <origin xyz="-0.25 -0.2 -0.22" rpy="0 0 0" />
                 <mass value="4"/>
                 <sphere_inertia m="${4}" r="${0.04}"/>
@@ -322,5 +322,5 @@
             <gravity>1</gravity>
             <collision name="sphere">
-                <origin xyz="-0.25 0 -0.21" rpy="0 0 0"/>
+                <origin xyz="-0.25 0 -0.22" rpy="0 0 0"/>
                 <geometry>
                     <sphere radius="0.03"/>
@@ -328,5 +328,5 @@
             </collision>
             <visual>
-                <origin xyz="-0.25 0 -0.21" rpy="0 0 0"/>
+                <origin xyz="-0.25 0 -0.22" rpy="0 0 0"/>
                 <geometry>
                     <sphere radius="0.03"/>
@@ -340,7 +340,7 @@
             </visual>
             <visual>
-                <origin xyz="-0.25 0 -0.175" rpy="0 0 0"/>
-                <geometry>
-                    <cylinder radius="0.007" length="0.055"/>
+                <origin xyz="-0.25 0 -0.18" rpy="0 0 0"/>
+                <geometry>
+                    <cylinder radius="0.007" length="0.065"/>
                 </geometry>
             </visual>
@@ -348,5 +348,5 @@
         <link name="tool3">
             <inertial>
-                <origin xyz="-0.25 0 -0.21" rpy="0 0 0" />
+                <origin xyz="-0.25 0 -0.22" rpy="0 0 0" />
                 <mass value="4"/>
                 <sphere_inertia m="${4}" r="${0.04}"/>
@@ -354,5 +354,5 @@
             <gravity>1</gravity>
             <collision name="sphere">
-                <origin xyz="-0.25 0 -0.21" rpy="0 0 0"/>
+                <origin xyz="-0.25 0 -0.22" rpy="0 0 0"/>
                 <geometry>
                     <sphere radius="0.03"/>
@@ -360,5 +360,5 @@
             </collision>
             <visual>
-                <origin xyz="-0.25 0 -0.21" rpy="0 0 0"/>
+                <origin xyz="-0.25 0 -0.22" rpy="0 0 0"/>
                 <geometry>
                     <sphere radius="0.03"/>
@@ -372,7 +372,7 @@
             </visual>
             <visual>
-                <origin xyz="-0.25 0 -0.175" rpy="0 0 0"/>
-                <geometry>
-                    <cylinder radius="0.007" length="0.055"/>
+                <origin xyz="-0.25 0 -0.18" rpy="0 0 0"/>
+                <geometry>
+                    <cylinder radius="0.007" length="0.065"/>
                 </geometry>
             </visual>

Commit message: distortion in the cameras, test 1

File: oz440_description/urdf/macros.xacro (robot description, xacro)
@@ -25,5 +25,5 @@
     </xacro:macro>
     <!-- macro pour creer les centres  -->
-    <xacro:macro name="center" params="fb lr tX tY">
+    <xacro:macro name="centers" params="fb lr tX tY">
         <link name="${fb}_${lr}_center">
             <visual>
@@ -281,141 +281,141 @@
     </xacro:macro>
     <!-- macro pour l'outils -->
-    <xacro:macro name="tool_macro" params="parent">
-        <link name="tool1">
-            <inertial>
-                <origin xyz="-0.25 0 -0.22" rpy="0 0 0" />
-                <mass value="4"/>
-                <sphere_inertia m="${4}" r="${0.04}"/>
-            </inertial>
-            <gravity>1</gravity>
-            <collision name="sphere">
-                <origin xyz="-0.25 0 -0.22" rpy="0 0 0"/>
-                <geometry>
-                    <sphere radius="0.03"/>
-                </geometry>
-            </collision>
-            <visual>
-                <origin xyz="-0.25 0 -0.22" rpy="0 0 0"/>
-                <geometry>
-                    <sphere radius="0.03"/>
-                </geometry>
-            </visual>
-            <visual>
-                <origin xyz="-0.125 0 -0.075" rpy="0 1.03 0"/>
-                <geometry>
-                    <cylinder radius="0.007" length="0.30"/>
-                </geometry>
-            </visual>
-            <visual>
-                <origin xyz="-0.25 0 -0.18" rpy="0 0 0"/>
-                <geometry>
-                    <cylinder radius="0.007" length="0.065"/>
-                </geometry>
-            </visual>
-        </link>
-        <link name="tool2">
-            <inertial>
-                <origin xyz="-0.25 -0.2 -0.22" rpy="0 0 0" />
-                <mass value="4"/>
-                <sphere_inertia m="${4}" r="${0.04}"/>
-            </inertial>
-            <gravity>1</gravity>
-            <collision name="sphere">
-                <origin xyz="-0.25 0 -0.22" rpy="0 0 0"/>
-                <geometry>
-                    <sphere radius="0.03"/>
-                </geometry>
-            </collision>
-            <visual>
-                <origin xyz="-0.25 0 -0.22" rpy="0 0 0"/>
-                <geometry>
-                    <sphere radius="0.03"/>
-                </geometry>
-            </visual>
-            <visual>
-                <origin xyz="-0.125 0 -0.075" rpy="0 1.03 0"/>
-                <geometry>
-                    <cylinder radius="0.007" length="0.29"/>
-                </geometry>
-            </visual>
-            <visual>
-                <origin xyz="-0.25 0 -0.18" rpy="0 0 0"/>
-                <geometry>
-                    <cylinder radius="0.007" length="0.065"/>
-                </geometry>
-            </visual>
-        </link>
-        <link name="tool3">
-            <inertial>
-                <origin xyz="-0.25 0 -0.22" rpy="0 0 0" />
-                <mass value="4"/>
-                <sphere_inertia m="${4}" r="${0.04}"/>
-            </inertial>
-            <gravity>1</gravity>
-            <collision name="sphere">
-                <origin xyz="-0.25 0 -0.22" rpy="0 0 0"/>
-                <geometry>
-                    <sphere radius="0.03"/>
-                </geometry>
-            </collision>
-            <visual>
-                <origin xyz="-0.25 0 -0.22" rpy="0 0 0"/>
-                <geometry>
-                    <sphere radius="0.03"/>
-                </geometry>
-            </visual>
-            <visual>
-                <origin xyz="-0.125 0 -0.075" rpy="0 1.03 0"/>
-                <geometry>
-                    <cylinder radius="0.007" length="0.29"/>
-                </geometry>
-            </visual>
-            <visual>
-                <origin xyz="-0.25 0 -0.18" rpy="0 0 0"/>
-                <geometry>
-                    <cylinder radius="0.007" length="0.065"/>
-                </geometry>
-            </visual>
-        </link>
-        <gazebo reference="tool1">
-            <mu1 value="0.99"/>
-            <mu2 value="0.99"/>
-            <kp  value="1e+6" />
-            <kd  value="1.0" />
-            <fdir1 value="0 0 0"/>
-            <material> Gazebo/Grey </material>
-        </gazebo>
-        <gazebo reference="tool2">
-            <mu1 value="0.99"/>
-            <mu2 value="0.99"/>
-            <kp  value="1e+6" />
-            <kd  value="1.0" />
-            <fdir1 value="0 0 0"/>
-            <material> Gazebo/Grey </material>
-        </gazebo>
-        <gazebo reference="tool3">
-            <mu1 value="0.99"/>
-            <mu2 value="0.99"/>
-            <kp  value="1e+6" />
-            <kd  value="1.0" />
-            <fdir1 value="0 0 0"/>
-            <material> Gazebo/Grey </material>
-        </gazebo>
-        <joint name="tool1_to_actuator_part_21" type="fixed">
-            <parent link="actuator_part21_link"/>
-            <child link="tool1"/>
-            <origin rpy="0 0 ${-actuator_part2_Height/2}" xyz="0 0 0"/>
-        </joint>
-        <joint name="tool2_to_actuator_part_22" type="fixed">
-            <parent link="actuator_part22_link"/>
-            <child link="tool2"/>
-            <origin rpy="0 0 ${-actuator_part2_Height/2}" xyz="0 0 0"/>
-        </joint>
-        <joint name="tool3_to_actuator_part_23" type="fixed">
-            <parent link="actuator_part23_link"/>
-            <child link="tool3"/>
-            <origin rpy="0 0 ${-actuator_part2_Height/2}" xyz="0 0 0"/>
-        </joint>
-    </xacro:macro>
+    <!--<xacro:macro name="tool_macro" params="parent">-->
+        <!--<link name="tool1">-->
+            <!--<inertial>-->
+                <!--<origin xyz="-0.25 0 -0.22" rpy="0 0 0" />-->
+                <!--<mass value="4"/>-->
+                <!--<sphere_inertia m="${4}" r="${0.04}"/>-->
+            <!--</inertial>-->
+            <!--<gravity>1</gravity>-->
+            <!--<collision name="sphere">-->
+                <!--<origin xyz="-0.25 0 -0.22" rpy="0 0 0"/>-->
+                <!--<geometry>-->
+                    <!--<sphere radius="0.03"/>-->
+                <!--</geometry>-->
+            <!--</collision>-->
+            <!--<visual>-->
+                <!--<origin xyz="-0.25 0 -0.22" rpy="0 0 0"/>-->
+                <!--<geometry>-->
+                    <!--<sphere radius="0.03"/>-->
+                <!--</geometry>-->
+            <!--</visual>-->
+            <!--<visual>-->
+                <!--<origin xyz="-0.125 0 -0.075" rpy="0 1.03 0"/>-->
+                <!--<geometry>-->
+                    <!--<cylinder radius="0.007" length="0.30"/>-->
+                <!--</geometry>-->
+            <!--</visual>-->
+            <!--<visual>-->
+                <!--<origin xyz="-0.25 0 -0.18" rpy="0 0 0"/>-->
+                <!--<geometry>-->
+                    <!--<cylinder radius="0.007" length="0.065"/>-->
+                <!--</geometry>-->
+            <!--</visual>-->
+        <!--</link>-->
+        <!--<link name="tool2">-->
+            <!--<inertial>-->
+                <!--<origin xyz="-0.25 -0.2 -0.22" rpy="0 0 0" />-->
+                <!--<mass value="4"/>-->
+                <!--<sphere_inertia m="${4}" r="${0.04}"/>-->
+            <!--</inertial>-->
+            <!--<gravity>1</gravity>-->
+            <!--<collision name="sphere">-->
+                <!--<origin xyz="-0.25 0 -0.22" rpy="0 0 0"/>-->
+                <!--<geometry>-->
+                    <!--<sphere radius="0.03"/>-->
+                <!--</geometry>-->
+            <!--</collision>-->
+            <!--<visual>-->
+                <!--<origin xyz="-0.25 0 -0.22" rpy="0 0 0"/>-->
+                <!--<geometry>-->
+                    <!--<sphere radius="0.03"/>-->
+                <!--</geometry>-->
+            <!--</visual>-->
+            <!--<visual>-->
+                <!--<origin xyz="-0.125 0 -0.075" rpy="0 1.03 0"/>-->
+                <!--<geometry>-->
+                    <!--<cylinder radius="0.007" length="0.29"/>-->
+                <!--</geometry>-->
+            <!--</visual>-->
+            <!--<visual>-->
+                <!--<origin xyz="-0.25 0 -0.18" rpy="0 0 0"/>-->
+                <!--<geometry>-->
+                    <!--<cylinder radius="0.007" length="0.065"/>-->
+                <!--</geometry>-->
+            <!--</visual>-->
+        <!--</link>-->
+        <!--<link name="tool3">-->
+            <!--<inertial>-->
+                <!--<origin xyz="-0.25 0 -0.22" rpy="0 0 0" />-->
+                <!--<mass value="4"/>-->
+                <!--<sphere_inertia m="${4}" r="${0.04}"/>-->
+            <!--</inertial>-->
+            <!--<gravity>1</gravity>-->
+            <!--<collision name="sphere">-->
+                <!--<origin xyz="-0.25 0 -0.22" rpy="0 0 0"/>-->
+                <!--<geometry>-->
+                    <!--<sphere radius="0.03"/>-->
+                <!--</geometry>-->
+            <!--</collision>-->
+            <!--<visual>-->
+                <!--<origin xyz="-0.25 0 -0.22" rpy="0 0 0"/>-->
+                <!--<geometry>-->
+                    <!--<sphere radius="0.03"/>-->
+                <!--</geometry>-->
+            <!--</visual>-->
+            <!--<visual>-->
+                <!--<origin xyz="-0.125 0 -0.075" rpy="0 1.03 0"/>-->
+                <!--<geometry>-->
+                    <!--<cylinder radius="0.007" length="0.29"/>-->
+                <!--</geometry>-->
+            <!--</visual>-->
+            <!--<visual>-->
+                <!--<origin xyz="-0.25 0 -0.18" rpy="0 0 0"/>-->
+                <!--<geometry>-->
+                    <!--<cylinder radius="0.007" length="0.065"/>-->
+                <!--</geometry>-->
+            <!--</visual>-->
+        <!--</link>-->
+        <!--<gazebo reference="tool1">-->
+            <!--<mu1 value="0.99"/>-->
+            <!--<mu2 value="0.99"/>-->
+            <!--<kp  value="1e+6" />-->
+            <!--<kd  value="1.0" />-->
+            <!--<fdir1 value="0 0 0"/>-->
+            <!--<material> Gazebo/Grey </material>-->
+        <!--</gazebo>-->
+        <!--<gazebo reference="tool2">-->
+            <!--<mu1 value="0.99"/>-->
+            <!--<mu2 value="0.99"/>-->
+            <!--<kp  value="1e+6" />-->
+            <!--<kd  value="1.0" />-->
+            <!--<fdir1 value="0 0 0"/>-->
+            <!--<material> Gazebo/Grey </material>-->
+        <!--</gazebo>-->
+        <!--<gazebo reference="tool3">-->
+            <!--<mu1 value="0.99"/>-->
+            <!--<mu2 value="0.99"/>-->
+            <!--<kp  value="1e+6" />-->
+            <!--<kd  value="1.0" />-->
+            <!--<fdir1 value="0 0 0"/>-->
+            <!--<material> Gazebo/Grey </material>-->
+        <!--</gazebo>-->
+        <!--<joint name="tool1_to_actuator_part_21" type="fixed">-->
+            <!--<parent link="actuator_part21_link"/>-->
+            <!--<child link="tool1"/>-->
+            <!--<origin rpy="0 0 ${-actuator_part2_Height/2}" xyz="0 0 0"/>-->
+        <!--</joint>-->
+        <!--<joint name="tool2_to_actuator_part_22" type="fixed">-->
+            <!--<parent link="actuator_part22_link"/>-->
+            <!--<child link="tool2"/>-->
+            <!--<origin rpy="0 0 ${-actuator_part2_Height/2}" xyz="0 0 0"/>-->
+        <!--</joint>-->
+        <!--<joint name="tool3_to_actuator_part_23" type="fixed">-->
+            <!--<parent link="actuator_part23_link"/>-->
+            <!--<child link="tool3"/>-->
+            <!--<origin rpy="0 0 ${-actuator_part2_Height/2}" xyz="0 0 0"/>-->
+        <!--</joint>-->
+    <!--</xacro:macro>-->
     <!-- macro pour la camera stereo -->
     <xacro:macro name="camera_stereo" params="parent">

File: oz440_description/urdf/oz440.xacro (robot description, xacro)
@@ -70,8 +70,8 @@
 	<wheel fb="back" lr="left" tX="-1" tY="1"/>
 	<!-- inclusion des roues -->
-	<center fb="front" lr="right" tX="1" tY="-1"/>
-	<center fb="front" lr="left" tX="1" tY="1"/>
-	<center fb="back" lr="right" tX="-1" tY="-1"/>
-	<center fb="back" lr="left" tX="-1" tY="1"/>
+	<centers fb="front" lr="right" tX="1" tY="-1"/>
+	<centers fb="front" lr="left" tX="1" tY="1"/>
+	<centers fb="back" lr="right" tX="-1" tY="-1"/>
+	<centers fb="back" lr="left" tX="-1" tY="1"/>
 	<!-- inclusion de la camera stereo -->
 	<camera_stereo parent="chassis_bottom"/>

Commit message: lidar bas

File: oz440_description/urdf/macros.xacro (robot description, xacro)
@@ -477,5 +477,5 @@
             <parent link="${parent}"/>
             <child link="lidar_link"/>
-            <origin xyz="${chassis_bottom_length/2+lidar_Lenght/2} 0 ${-chassis_bottom_height/2-lidar_chassis_bottom_spacing+lidar_Height/2}" rpy="0 0 0"/>
+            <origin xyz="${chassis_bottom_length/2+lidar_Lenght/2} 0 ${-chassis_bottom_height/2-lidar_chassis_bottom_spacing+lidar_Height/2 -0.06}" rpy="0 0 0"/>
         </joint>
     </xacro:macro>

File: oz440_description/urdf/oz440.xacro (robot description, xacro)
@@ -63,5 +63,5 @@
 	<!-- inclusion du porte outils -->
     <actuator_macro parent="chassis_bottom"/>
-	<tool_macro parent="actuator_part2_link"/>
+	<!--<tool_macro parent="actuator_part2_link"/>-->
     <!-- inclusion des roues -->
 	<wheel fb="front" lr="right" tX="1" tY="-1"/>

Commit message: Ok sans tool

File: oz440_description/urdf/macros.xacro (robot description, xacro)
@@ -477,5 +477,5 @@
             <parent link="${parent}"/>
             <child link="lidar_link"/>
-            <origin xyz="${chassis_bottom_length/2+lidar_Lenght/2} 0 ${-chassis_bottom_height/2-lidar_chassis_bottom_spacing+lidar_Height/2 -0.06}" rpy="0 0 0"/>
+            <origin xyz="${chassis_bottom_length/2+lidar_Lenght/2} 0 ${-chassis_bottom_height/2-lidar_chassis_bottom_spacing+lidar_Height/2}" rpy="0 0 0"/>
         </joint>
     </xacro:macro>
