Commit message: distort _image function

File: oz440_description/urdf/macros.xacro (robot description, xacro)
@@ -82,5 +82,5 @@
             <mu1 value="0.99"/>
             <mu2 value="0.99"/>
-            <kp  value="1e+7" />
+            <kp  value="1e+60" />
             <kd  value="1.0" />
             <material>Gazebo/DarkGrey</material>
@@ -280,142 +280,142 @@
         </joint>
     </xacro:macro>
-    <!-- macro pour l'outils -->
-    <!--<xacro:macro name="tool_macro" params="parent">-->
-        <!--<link name="tool1">-->
-            <!--<inertial>-->
-                <!--<origin xyz="-0.25 0 -0.22" rpy="0 0 0" />-->
-                <!--<mass value="4"/>-->
-                <!--<sphere_inertia m="${4}" r="${0.04}"/>-->
-            <!--</inertial>-->
-            <!--<gravity>1</gravity>-->
-            <!--<collision name="sphere">-->
-                <!--<origin xyz="-0.25 0 -0.22" rpy="0 0 0"/>-->
-                <!--<geometry>-->
-                    <!--<sphere radius="0.03"/>-->
-                <!--</geometry>-->
-            <!--</collision>-->
-            <!--<visual>-->
-                <!--<origin xyz="-0.25 0 -0.22" rpy="0 0 0"/>-->
-                <!--<geometry>-->
-                    <!--<sphere radius="0.03"/>-->
-                <!--</geometry>-->
-            <!--</visual>-->
-            <!--<visual>-->
-                <!--<origin xyz="-0.125 0 -0.075" rpy="0 1.03 0"/>-->
-                <!--<geometry>-->
-                    <!--<cylinder radius="0.007" length="0.30"/>-->
-                <!--</geometry>-->
-            <!--</visual>-->
-            <!--<visual>-->
-                <!--<origin xyz="-0.25 0 -0.18" rpy="0 0 0"/>-->
-                <!--<geometry>-->
-                    <!--<cylinder radius="0.007" length="0.065"/>-->
-                <!--</geometry>-->
-            <!--</visual>-->
-        <!--</link>-->
-        <!--<link name="tool2">-->
-            <!--<inertial>-->
-                <!--<origin xyz="-0.25 -0.2 -0.22" rpy="0 0 0" />-->
-                <!--<mass value="4"/>-->
-                <!--<sphere_inertia m="${4}" r="${0.04}"/>-->
-            <!--</inertial>-->
-            <!--<gravity>1</gravity>-->
-            <!--<collision name="sphere">-->
-                <!--<origin xyz="-0.25 0 -0.22" rpy="0 0 0"/>-->
-                <!--<geometry>-->
-                    <!--<sphere radius="0.03"/>-->
-                <!--</geometry>-->
-            <!--</collision>-->
-            <!--<visual>-->
-                <!--<origin xyz="-0.25 0 -0.22" rpy="0 0 0"/>-->
-                <!--<geometry>-->
-                    <!--<sphere radius="0.03"/>-->
-                <!--</geometry>-->
-            <!--</visual>-->
-            <!--<visual>-->
-                <!--<origin xyz="-0.125 0 -0.075" rpy="0 1.03 0"/>-->
-                <!--<geometry>-->
-                    <!--<cylinder radius="0.007" length="0.29"/>-->
-                <!--</geometry>-->
-            <!--</visual>-->
-            <!--<visual>-->
-                <!--<origin xyz="-0.25 0 -0.18" rpy="0 0 0"/>-->
-                <!--<geometry>-->
-                    <!--<cylinder radius="0.007" length="0.065"/>-->
-                <!--</geometry>-->
-            <!--</visual>-->
-        <!--</link>-->
-        <!--<link name="tool3">-->
-            <!--<inertial>-->
-                <!--<origin xyz="-0.25 0 -0.22" rpy="0 0 0" />-->
-                <!--<mass value="4"/>-->
-                <!--<sphere_inertia m="${4}" r="${0.04}"/>-->
-            <!--</inertial>-->
-            <!--<gravity>1</gravity>-->
-            <!--<collision name="sphere">-->
-                <!--<origin xyz="-0.25 0 -0.22" rpy="0 0 0"/>-->
-                <!--<geometry>-->
-                    <!--<sphere radius="0.03"/>-->
-                <!--</geometry>-->
-            <!--</collision>-->
-            <!--<visual>-->
-                <!--<origin xyz="-0.25 0 -0.22" rpy="0 0 0"/>-->
-                <!--<geometry>-->
-                    <!--<sphere radius="0.03"/>-->
-                <!--</geometry>-->
-            <!--</visual>-->
-            <!--<visual>-->
-                <!--<origin xyz="-0.125 0 -0.075" rpy="0 1.03 0"/>-->
-                <!--<geometry>-->
-                    <!--<cylinder radius="0.007" length="0.29"/>-->
-                <!--</geometry>-->
-            <!--</visual>-->
-            <!--<visual>-->
-                <!--<origin xyz="-0.25 0 -0.18" rpy="0 0 0"/>-->
-                <!--<geometry>-->
-                    <!--<cylinder radius="0.007" length="0.065"/>-->
-                <!--</geometry>-->
-            <!--</visual>-->
-        <!--</link>-->
-        <!--<gazebo reference="tool1">-->
-            <!--<mu1 value="0.99"/>-->
-            <!--<mu2 value="0.99"/>-->
-            <!--<kp  value="1e+6" />-->
-            <!--<kd  value="1.0" />-->
-            <!--<fdir1 value="0 0 0"/>-->
-            <!--<material> Gazebo/Grey </material>-->
-        <!--</gazebo>-->
-        <!--<gazebo reference="tool2">-->
-            <!--<mu1 value="0.99"/>-->
-            <!--<mu2 value="0.99"/>-->
-            <!--<kp  value="1e+6" />-->
-            <!--<kd  value="1.0" />-->
-            <!--<fdir1 value="0 0 0"/>-->
-            <!--<material> Gazebo/Grey </material>-->
-        <!--</gazebo>-->
-        <!--<gazebo reference="tool3">-->
-            <!--<mu1 value="0.99"/>-->
-            <!--<mu2 value="0.99"/>-->
-            <!--<kp  value="1e+6" />-->
-            <!--<kd  value="1.0" />-->
-            <!--<fdir1 value="0 0 0"/>-->
-            <!--<material> Gazebo/Grey </material>-->
-        <!--</gazebo>-->
-        <!--<joint name="tool1_to_actuator_part_21" type="fixed">-->
-            <!--<parent link="actuator_part21_link"/>-->
-            <!--<child link="tool1"/>-->
-            <!--<origin rpy="0 0 ${-actuator_part2_Height/2}" xyz="0 0 0"/>-->
-        <!--</joint>-->
-        <!--<joint name="tool2_to_actuator_part_22" type="fixed">-->
-            <!--<parent link="actuator_part22_link"/>-->
-            <!--<child link="tool2"/>-->
-            <!--<origin rpy="0 0 ${-actuator_part2_Height/2}" xyz="0 0 0"/>-->
-        <!--</joint>-->
-        <!--<joint name="tool3_to_actuator_part_23" type="fixed">-->
-            <!--<parent link="actuator_part23_link"/>-->
-            <!--<child link="tool3"/>-->
-            <!--<origin rpy="0 0 ${-actuator_part2_Height/2}" xyz="0 0 0"/>-->
-        <!--</joint>-->
-    <!--</xacro:macro>-->
+     <!--macro pour l'outils-->
+    <xacro:macro name="tool_macro" params="parent">
+        <link name="tool1">
+            <inertial>
+                <origin xyz="-0.25 0 -0.22" rpy="0 0 0" />
+                <mass value="4"/>
+                <sphere_inertia m="${4}" r="${0.04}"/>
+            </inertial>
+            <gravity>1</gravity>
+            <collision name="sphere">
+                <origin xyz="-0.25 0 -0.22" rpy="0 0 0"/>
+                <geometry>
+                    <sphere radius="0.03"/>
+                </geometry>
+            </collision>
+            <visual>
+                <origin xyz="-0.25 0 -0.22" rpy="0 0 0"/>
+                <geometry>
+                    <sphere radius="0.03"/>
+                </geometry>
+            </visual>
+            <visual>
+                <origin xyz="-0.125 0 -0.075" rpy="0 1.03 0"/>
+                <geometry>
+                    <cylinder radius="0.007" length="0.30"/>
+                </geometry>
+            </visual>
+            <visual>
+                <origin xyz="-0.25 0 -0.18" rpy="0 0 0"/>
+                <geometry>
+                    <cylinder radius="0.007" length="0.065"/>
+                </geometry>
+            </visual>
+        </link>
+        <link name="tool2">
+            <inertial>
+                <origin xyz="-0.25 -0.2 -0.22" rpy="0 0 0" />
+                <mass value="4"/>
+                <sphere_inertia m="${4}" r="${0.04}"/>
+            </inertial>
+            <gravity>1</gravity>
+            <collision name="sphere">
+                <origin xyz="-0.25 0 -0.22" rpy="0 0 0"/>
+                <geometry>
+                    <sphere radius="0.03"/>
+                </geometry>
+            </collision>
+            <visual>
+                <origin xyz="-0.25 0 -0.22" rpy="0 0 0"/>
+                <geometry>
+                    <sphere radius="0.03"/>
+                </geometry>
+            </visual>
+            <visual>
+                <origin xyz="-0.125 0 -0.075" rpy="0 1.03 0"/>
+                <geometry>
+                    <cylinder radius="0.007" length="0.29"/>
+                </geometry>
+            </visual>
+            <visual>
+                <origin xyz="-0.25 0 -0.18" rpy="0 0 0"/>
+                <geometry>
+                    <cylinder radius="0.007" length="0.065"/>
+                </geometry>
+            </visual>
+        </link>
+        <link name="tool3">
+            <inertial>
+                <origin xyz="-0.25 0 -0.22" rpy="0 0 0" />
+                <mass value="4"/>
+                <sphere_inertia m="${4}" r="${0.04}"/>
+            </inertial>
+            <gravity>1</gravity>
+            <collision name="sphere">
+                <origin xyz="-0.25 0 -0.22" rpy="0 0 0"/>
+                <geometry>
+                    <sphere radius="0.03"/>
+                </geometry>
+            </collision>
+            <visual>
+                <origin xyz="-0.25 0 -0.22" rpy="0 0 0"/>
+                <geometry>
+                    <sphere radius="0.03"/>
+                </geometry>
+            </visual>
+            <visual>
+                <origin xyz="-0.125 0 -0.075" rpy="0 1.03 0"/>
+                <geometry>
+                    <cylinder radius="0.007" length="0.29"/>
+                </geometry>
+            </visual>
+            <visual>
+                <origin xyz="-0.25 0 -0.18" rpy="0 0 0"/>
+                <geometry>
+                    <cylinder radius="0.007" length="0.065"/>
+                </geometry>
+            </visual>
+        </link>
+        <gazebo reference="tool1">
+            <mu1 value="0.99"/>
+            <mu2 value="0.99"/>
+            <kp  value="1e+6" />
+            <kd  value="1.0" />
+            <fdir1 value="0 0 0"/>
+            <material> Gazebo/Grey </material>
+        </gazebo>
+        <gazebo reference="tool2">
+            <mu1 value="0.99"/>
+            <mu2 value="0.99"/>
+            <kp  value="1e+6" />
+            <kd  value="1.0" />
+            <fdir1 value="0 0 0"/>
+            <material> Gazebo/Grey </material>
+        </gazebo>
+        <gazebo reference="tool3">
+            <mu1 value="0.99"/>
+            <mu2 value="0.99"/>
+            <kp  value="1e+6" />
+            <kd  value="1.0" />
+            <fdir1 value="0 0 0"/>
+            <material> Gazebo/Grey </material>
+        </gazebo>
+        <joint name="tool1_to_actuator_part_21" type="fixed">
+            <parent link="actuator_part21_link"/>
+            <child link="tool1"/>
+            <origin rpy="0 0 ${-actuator_part2_Height/2}" xyz="0 0 0"/>
+        </joint>
+        <joint name="tool2_to_actuator_part_22" type="fixed">
+            <parent link="actuator_part22_link"/>
+            <child link="tool2"/>
+            <origin rpy="0 0 ${-actuator_part2_Height/2}" xyz="0 0 0"/>
+        </joint>
+        <joint name="tool3_to_actuator_part_23" type="fixed">
+            <parent link="actuator_part23_link"/>
+            <child link="tool3"/>
+            <origin rpy="0 0 ${-actuator_part2_Height/2}" xyz="0 0 0"/>
+        </joint>
+    </xacro:macro>
     <!-- macro pour la camera stereo -->
     <xacro:macro name="camera_stereo" params="parent">

File: oz440_description/urdf/oz440.xacro (robot description, xacro)
@@ -63,4 +63,5 @@
 	<!-- inclusion du porte outils -->
     <actuator_macro parent="chassis_bottom"/>
+	<!-- inclusion de l'outil -->
 	<!--<tool_macro parent="actuator_part2_link"/>-->
     <!-- inclusion des roues -->

Commit message: new worlds

File: oz440_description/urdf/macros.xacro (robot description, xacro)
@@ -80,8 +80,9 @@
         <gazebo reference="${fb}_${lr}_wheel">
             <gravity>true</gravity>
-            <mu1 value="0.99"/>
-            <mu2 value="0.99"/>
-            <kp  value="1e+7" />
-            <kd  value="1.0" />
+            <mu1 value="10"/>
+            <mu2 value="10"/>
+            <kp  value="1e+7" />
+            <kd  value="100.0" />
+            <!--<fdir1 value="0 1 0"/>-->
             <material>Gazebo/DarkGrey</material>
         </gazebo>

File: oz440_description/urdf/properties.xacro (robot description, xacro)
@@ -10,5 +10,5 @@
 	<!-- Proprietes de la partie haute du robot -->
 	<xacro:property name="chassis_top_height" value="0.220"/>
-	<xacro:property name="chassis_top_width" value="0.41389"/>
+	<xacro:property name="chassis_top_width" value="0.42"/>
 	<xacro:property name="chassis_top_length" value="0.67454"/>
 	<xacro:property name="chassis_top_mass" value="70"/>
@@ -18,5 +18,5 @@
 	<xacro:property name="wheel_width" value="0.08761"/>
 	<xacro:property name="wheel_transmission_height" value="0.058"/>
-	<xacro:property name="wheel_chassis_bottom_spacing" value="0.01"/>
+	<xacro:property name="wheel_chassis_bottom_spacing" value="0.025"/>
 	<xacro:property name="wheels_spacing" value="0.435"/>
 	<xacro:property name="wheel_mass" value="3"/>
